File: hardware/ButterStick/SYZYGY_PORT2.sch (KiCad schematic (older format))
At the start: 2 parts, among them U3 ECP5U25

Commit message: Routed all SYZYGY ports. Placed decoupling caps etc.
Parts:
- R28: footprint (none) -> pkl_dipol:R_0402
- U3: footprint (none) -> gkl_housings_bga:caBGA_381_17x17
Connections:
- net S16: now also U3.L2 (PL41D); no longer U3.L5 (PL35D)
- net S17: now also U3.P3 (PL47C/LLC_GPLL0T_IN); no longer U3.N4 (PL38C)
- net S18: now also U3.L5 (PL35D); no longer U3.L2 (PL41D)
- net S19: now also U3.P4 (PL47D/LLC_GPLL0C_IN); no longer U3.P5 (PL38D)
- net S20: now also U3.L4 (PL35C); no longer U3.L1 (PL44C)
- net S22: now also U3.P5 (PL38D); no longer U3.N1 (PL44D)
- net S24: now also U3.N4 (PL38C); no longer U3.P3 (PL47C/LLC_GPLL0T_IN)
- net S25: now also U3.K1 (PL32D); no longer U3.L4 (PL35C)
- net S26: now also U3.N1 (PL44D); no longer U3.P4 (PL47D/LLC_GPLL0C_IN)
- net S27: now also U3.L1 (PL44C); no longer U3.K1 (PL32D)
Changed lines of the file:
@@
 $Descr A4 11693 8268
 encoding utf-8
-Sheet 12 13
+Sheet 12 14
 Title ""
 Date ""
@@
 F 0 "U3" H 5500 2650 60  0000 L CNN
 F 1 "ECP5U25" H 4600 2650 60  0000 L CNN
-F 2 "" H 4400 2450 50  0001 C CNN
+F 2 "gkl_housings_bga:caBGA_381_17x17" H 4400 2450 50  0001 C CNN
 F 3 "" H 4400 2450 50  0001 C CNN
 F 4 " 220-2052-ND " H -1850 -1950 50  0001 C CNN "SN-DK"
@@
 C2P_CLK_N
 Wire Wire Line
+	4400 4750 4850 4750
+Wire Wire Line
+	4400 5450 4850 5450
+Wire Wire Line
 	4400 3950 4850 3950
 Wire Wire Line
+	4400 5550 4850 5550
+Wire Wire Line
+	4400 3850 4850 3850
+Wire Wire Line
+	4400 3450 4850 3450
+Wire Wire Line
+	4400 4350 4850 4350
+Wire Wire Line
+	4400 4650 4850 4650
+Wire Wire Line
 	4400 4250 4850 4250
 Wire Wire Line
-	4400 4750 4850 4750
-Wire Wire Line
-	4400 4350 4850 4350
+	4400 3550 4850 3550
+Wire Wire Line
+	4400 5150 4850 5150
 Wire Wire Line
 	4400 5050 4850 5050
 Wire Wire Line
-	4400 3450 4850 3450
-Wire Wire Line
-	4400 5150 4850 5150
-Wire Wire Line
-	4400 4650 4850 4650
-Wire Wire Line
-	4400 5450 4850 5450
-Wire Wire Line
-	4400 3850 4850 3850
-Wire Wire Line
-	4400 5550 4850 5550
-Wire Wire Line
-	4400 3550 4850 3550
-Wire Wire Line
 	4400 2850 5050 2850
 Wire Wire Line
@@
 Wire Wire Line
 	4400 2550 5350 2550
+Text Label 4850 4750 2    50   ~ 0
+S16
+Text Label 4850 5450 2    50   ~ 0
+S17
 Text Label 4850 3950 2    50   ~ 0
-S16
-Text Label 4850 4250 2    50   ~ 0
-S17
-Text Label 4850 4750 2    50   ~ 0
 S18
-Text Label 4850 4350 2    50   ~ 0
+Text Label 4850 5550 2    50   ~ 0
 S19
-Text Label 4850 5050 2    50   ~ 0
+Text Label 4850 3850 2    50   ~ 0
 S20
 Text Label 4850 3450 2    50   ~ 0
 S21
-Text Label 4850 5150 2    50   ~ 0
+Text Label 4850 4350 2    50   ~ 0
 S22
 Text Label 4850 4650 2    50   ~ 0
 S23
-Text Label 4850 5450 2    50   ~ 0
+Text Label 4850 4250 2    50   ~ 0
 S24
-Text Label 4850 3850 2    50   ~ 0
+Text Label 4850 3550 2    50   ~ 0
 S25
-Text Label 4850 5550 2    50   ~ 0
+Text Label 4850 5150 2    50   ~ 0
 S26
-Text Label 4850 3550 2    50   ~ 0
+Text Label 4850 5050 2    50   ~ 0
 S27
 Text Label 5050 2850 2    50   ~ 0
@@
 F 0 "R28" H 9020 3746 50  0000 L CNN
 F 1 "R" H 9020 3655 50  0000 L CNN
-F 2 "" V 8880 3700 50  0001 C CNN
+F 2 "pkl_dipol:R_0402" V 8880 3700 50  0001 C CNN
 F 3 "~" H 8950 3700 50  0001 C CNN
 	1    8950 3700

Commit message: Added ESD on SD card signals.
Connections:
- no-connect marks 0 -> 1
Changed lines of the file:
@@
 $Descr A4 11693 8268
 encoding utf-8
-Sheet 12 14
+Sheet 12 13
 Title ""
 Date ""
@@
 	1    0    0    -1
 $EndComp
-$Comp
-L gkl_power:GND #PWR0217
-U 1 1 5C987095
-P 9350 3150
-F 0 "#PWR0217" H 9350 2900 50  0001 C CNN
-F 1 "GND" V 9354 3070 50  0000 R CNN
-F 2 "" H 9250 2800 50  0001 C CNN
-F 3 "" H 9350 3150 50  0001 C CNN
-	1    9350 3150
-	0    -1   -1   0
-$EndComp
-Wire Wire Line
-	8700 3150 9350 3150
 Wire Wire Line
 	8700 2350 9100 2350
@@
 Text HLabel 9100 2950 2    50   Input ~ 0
 pmicSDA
+NoConn ~ 8700 3150
 $EndSCHEMATC

Commit message: Finished initial routing of PCB.. Most parts are finished.
Changed lines of the file:
@@
 $Descr A4 11693 8268
 encoding utf-8
-Sheet 12 13
+Sheet 11 13
 Title ""
 Date ""
@@
 F39 "VCCIO" I R 8700 2350 50
 F40 "R_GA" I R 8700 3250 50
+F41 "PMIC_EN" I R 8700 2450 50
 $EndSheet
 Wire Wire Line
@@
 pmicSDA
 NoConn ~ 8700 3150
+Wire Wire Line
+	8700 2450 9100 2450
+Text HLabel 9100 2450 2    50   Input ~ 0
+EN
 $EndSCHEMATC

Commit message: Update KiCad PCB.
Parts:
- U3: PN LFE5U-25F-6BG381I -> LFE5U-45F-8BG381C
Changed lines of the file:
@@
 F 3 "" H 4400 2450 50  0001 C CNN
 F 4 " 220-2052-ND " H -1850 -1950 50  0001 C CNN "SN-DK"
-F 5 " LFE5U-25F-6BG381I " H -1850 -1950 50  0001 C CNN "PN"
+F 5 "LFE5U-45F-8BG381C" H -1850 -1950 50  0001 C CNN "PN"
 F 6 "Lattice" H -1850 -1950 50  0001 C CNN "Mfg"
 	5    4400 2450

Commit message: Finalised part values update BOM values to reflect. Swapped layers 4/5 due to stackup changes
Parts:
- R28: value R -> 49k9; Mfg (none) -> Stackpole Electronics Inc; PN (none) -> RMCF0402FT49K9; Tol (none) -> 1%
Changed lines of the file:
@@
 EESchema Schematic File Version 4
 LIBS:ButterStick-cache
-EELAYER 26 0
+EELAYER 29 0
 EELAYER END
 $Descr A4 11693 8268
 encoding utf-8
-Sheet 11 13
-Title ""
-Date ""
-Rev ""
-Comp ""
+Sheet 5 13
+Title "ButterStick"
+Date "2019-03-19"
+Rev "r0_1"
+Comp "GsD"
 Comment1 ""
 Comment2 ""
@@
 P 8950 3700
 F 0 "R28" H 9020 3746 50  0000 L CNN
-F 1 "R" H 9020 3655 50  0000 L CNN
+F 1 "49k9" H 9020 3655 50  0000 L CNN
 F 2 "pkl_dipol:R_0402" V 8880 3700 50  0001 C CNN
 F 3 "~" H 8950 3700 50  0001 C CNN
+F 4 "Stackpole Electronics Inc" H 0   0   50  0001 C CNN "Mfg"
+F 5 "RMCF0402FT49K9" H 0   0   50  0001 C CNN "PN"
+F 6 "1%" H 0   0   50  0001 C CNN "Tol"
 	1    8950 3700
 	1    0    0    -1
