File: hardware/ButterStick/filePower.sch (KiCad schematic (older format))
At the start: 57 parts, among them J6 JST_PA, U1 TLV725P, U15 TPS542951, U21 LTC4367, U22 AON7804, U8 TLV718P, U9 TLV711P

Commit message: Finalised part values update BOM values to reflect. Swapped layers 4/5 due to stackup changes
Parts:
- C11, C13, C14: PN C1608X5R1A106K080AC -> CL10A106MP8NNNC
- C3, C4, C5: Mfg (none) -> Samsung Electro-Mechanics; PN CGB2A1X5R1E105K033BC -> CL05A105KP5NNNC
- C51: Mfg (none) -> Samsung Electro-Mechanics; PN CL05B104KP5NNNC -> CL05A105KP5NNNC
- C52, C53, C54, C56: PN CL05B104KP5NNNC -> CL21A226MOCLRNC
- C57, C60: PN CL05B104KP5NNNC -> CL05C100JB5NNNC
- C58, C59: Mfg (none) -> Samsung Electro-Mechanics; PN CL05B104KP5NNNC -> CL05B103KB5NNNC
- C67, C69, C70: PN CL05B104KP5NNNC -> CL21A106KAFN3NE; SN-DK 1276-1002-1-ND -> (none)
- C68: PN CL05B104KP5NNNC -> CL10B104KB8NNNC; SN-DK 1276-1002-1-ND -> (none)
- J6: Mfg (none) -> JST Sales America Inc.; PN (none) -> S02B-PASK-2(LF)(SN)
- R43, R56, R57, R58: Mfg (none) -> Stackpole Electronics Inc; PN (none) -> RMCF0402FT124K
- R44, R46: Mfg (none) -> Stackpole Electronics Inc; PN (none) -> RMCF0402FT22K1
- R45: Mfg (none) -> Stackpole Electronics Inc; PN (none) -> RMCF0402FT73K2
- R59: Mfg (none) -> Stackpole Electronics Inc; PN (none) -> RMCF0402FT510K
- R61, R62: Mfg (none) -> Stackpole Electronics Inc; PN (none) -> RMCF0402FT10K0
Changed lines of the file:
@@
 EESchema Schematic File Version 4
 LIBS:ButterStick-cache
-EELAYER 26 0
+EELAYER 29 0
 EELAYER END
 $Descr A4 11693 8268
 encoding utf-8
-Sheet 6 13
-Title ""
-Date ""
-Rev ""
-Comp ""
+Sheet 11 13
+Title "ButterStick"
+Date "2019-03-19"
+Rev "r0_1"
+Comp "GsD"
 Comment1 ""
 Comment2 ""
@@
 F 3 "" H 3450 5200 50  0001 C CNN
 F 4 "445-13185-1-ND" H -150 -150 50  0001 C CNN "SN-DK"
-F 5 "CGB2A1X5R1E105K033BC" H -150 -150 50  0001 C CNN "PN"
+F 5 "CL05A105KP5NNNC" H -150 -150 50  0001 C CNN "PN"
+F 6 "Samsung Electro-Mechanics" H 0   0   50  0001 C CNN "Mfg"
 	1    3450 5200
 	1    0    0    -1
@@
 F 3 "" H 3450 5950 50  0001 C CNN
 F 4 "445-13185-1-ND" H -150 -150 50  0001 C CNN "SN-DK"
-F 5 "CGB2A1X5R1E105K033BC" H -150 -150 50  0001 C CNN "PN"
+F 5 "CL05A105KP5NNNC" H -150 -150 50  0001 C CNN "PN"
+F 6 "Samsung Electro-Mechanics" H 0   0   50  0001 C CNN "Mfg"
 	1    3450 5950
 	1    0    0    -1
@@
 F 3 "" H 10300 4500 50  0001 C CNN
 F 4 "445-7486-1-ND" H 9050 -850 50  0001 C CNN "SN-DK"
-F 5 "C1608X5R1A106K080AC" H 9050 -850 50  0001 C CNN "PN"
+F 5 "CL10A106MP8NNNC" H 0   0   50  0001 C CNN "PN"
 	1    10300 4500
 	1    0    0    -1
@@
 F 3 "" H 10700 4500 50  0001 C CNN
 F 4 "445-7486-1-ND" H 9050 -850 50  0001 C CNN "SN-DK"
-F 5 "C1608X5R1A106K080AC" H 9050 -850 50  0001 C CNN "PN"
+F 5 "CL10A106MP8NNNC" H 0   0   50  0001 C CNN "PN"
 	1    10700 4500
 	1    0    0    -1
@@
 F 3 "" H 9900 4500 50  0001 C CNN
 F 4 "445-7486-1-ND" H 9050 -850 50  0001 C CNN "SN-DK"
-F 5 "C1608X5R1A106K080AC" H 9050 -850 50  0001 C CNN "PN"
+F 5 "CL10A106MP8NNNC" H 0   0   50  0001 C CNN "PN"
 	1    9900 4500
 	1    0    0    -1
@@
 F 3 "" H 3450 6700 50  0001 C CNN
 F 4 "445-13185-1-ND" H -150 -150 50  0001 C CNN "SN-DK"
-F 5 "CGB2A1X5R1E105K033BC" H -150 -150 50  0001 C CNN "PN"
+F 5 "CL05A105KP5NNNC" H -150 -150 50  0001 C CNN "PN"
+F 6 "Samsung Electro-Mechanics" H 0   0   50  0001 C CNN "Mfg"
 	1    3450 6700
 	1    0    0    -1
@@
 F 3 "" H 7000 3550 50  0001 C CNN
 F 4 "1276-1002-1-ND" H 2500 -3400 50  0001 C CNN "SN-DK"
-F 5 "CL05B104KP5NNNC" H 2500 -3400 50  0001 C CNN "PN"
+F 5 "CL05A105KP5NNNC" H 2500 -3400 50  0001 C CNN "PN"
+F 6 "Samsung Electro-Mechanics" H 0   0   50  0001 C CNN "Mfg"
 	1    7000 3550
 	1    0    0    -1
@@
 F 3 "" H 5000 2800 50  0001 C CNN
 F 4 "1276-1002-1-ND" H 500 -4150 50  0001 C CNN "SN-DK"
-F 5 "CL05B104KP5NNNC" H 500 -4150 50  0001 C CNN "PN"
+F 5 "CL21A226MOCLRNC" H 0   0   50  0001 C CNN "PN"
 	1    5000 2800
 	1    0    0    -1
@@
 F 3 "" H 4700 2800 50  0001 C CNN
 F 4 "1276-1002-1-ND" H 200 -4150 50  0001 C CNN "SN-DK"
-F 5 "CL05B104KP5NNNC" H 200 -4150 50  0001 C CNN "PN"
+F 5 "CL21A226MOCLRNC" H 0   0   50  0001 C CNN "PN"
 	1    4700 2800
 	1    0    0    -1
@@
 F 3 "" H 7800 2800 50  0001 C CNN
 F 4 "1276-1002-1-ND" H 3300 -4150 50  0001 C CNN "SN-DK"
-F 5 "CL05B104KP5NNNC" H 3300 -4150 50  0001 C CNN "PN"
+F 5 "CL21A226MOCLRNC" H 0   0   50  0001 C CNN "PN"
 	1    7800 2800
 	-1   0    0    -1
@@
 F 3 "" H 8100 2800 50  0001 C CNN
 F 4 "1276-1002-1-ND" H 3600 -4150 50  0001 C CNN "SN-DK"
-F 5 "CL05B104KP5NNNC" H 3600 -4150 50  0001 C CNN "PN"
+F 5 "CL21A226MOCLRNC" H 0   0   50  0001 C CNN "PN"
 	1    8100 2800
 	-1   0    0    -1
@@
 F 2 "pkl_dipol:R_0402" V 4080 2950 50  0001 C CNN
 F 3 "~" H 4150 2950 50  0001 C CNN
+F 4 "Stackpole Electronics Inc" H 0   0   50  0001 C CNN "Mfg"
+F 5 "RMCF0402FT124K" H 0   0   50  0001 C CNN "PN"
 	1    4150 2950
 	1    0    0    -1
@@
 F 2 "pkl_dipol:R_0402" V 4080 3500 50  0001 C CNN
 F 3 "~" H 4150 3500 50  0001 C CNN
+F 4 "Stackpole Electronics Inc" H 0   0   50  0001 C CNN "Mfg"
+F 5 "RMCF0402FT22K1" H 0   0   50  0001 C CNN "PN"
 	1    4150 3500
 	1    0    0    -1
@@
 F 3 "" H 3900 2950 50  0001 C CNN
 F 4 "1276-1002-1-ND" H -600 -4000 50  0001 C CNN "SN-DK"
-F 5 "CL05B104KP5NNNC" H -600 -4000 50  0001 C CNN "PN"
+F 5 "CL05C100JB5NNNC" H 0   0   50  0001 C CNN "PN"
 	1    3900 2950
 	1    0    0    -1
@@
 F 3 "" H 5350 3500 50  0001 C CNN
 F 4 "1276-1002-1-ND" H 850 -3450 50  0001 C CNN "SN-DK"
-F 5 "CL05B104KP5NNNC" H 850 -3450 50  0001 C CNN "PN"
+F 5 "CL05B103KB5NNNC" H 850 -3450 50  0001 C CNN "PN"
+F 6 "Samsung Electro-Mechanics" H 0   0   50  0001 C CNN "Mfg"
 	1    5350 3500
 	1    0    0    -1
@@
 F 3 "" H 7450 3550 50  0001 C CNN
 F 4 "1276-1002-1-ND" H 2950 -3400 50  0001 C CNN "SN-DK"
-F 5 "CL05B104KP5NNNC" H 2950 -3400 50  0001 C CNN "PN"
+F 5 "CL05B103KB5NNNC" H 2950 -3400 50  0001 C CNN "PN"
+F 6 "Samsung Electro-Mechanics" H 0   0   50  0001 C CNN "Mfg"
 	1    7450 3550
 	1    0    0    -1
@@
 F 2 "pkl_dipol:R_0402" V 8580 2950 50  0001 C CNN
 F 3 "~" H 8650 2950 50  0001 C CNN
+F 4 "Stackpole Electronics Inc" H 0   0   50  0001 C CNN "Mfg"
+F 5 "RMCF0402FT73K2" H 0   0   50  0001 C CNN "PN"
 	1    8650 2950
 	-1   0    0    -1
@@
 F 2 "pkl_dipol:R_0402" V 8580 3500 50  0001 C CNN
 F 3 "~" H 8650 3500 50  0001 C CNN
+F 4 "Stackpole Electronics Inc" H 0   0   50  0001 C CNN "Mfg"
+F 5 "RMCF0402FT22K1" H 0   0   50  0001 C CNN "PN"
 	1    8650 3500
 	-1   0    0    -1
@@
 F 3 "" H 8900 2950 50  0001 C CNN
 F 4 "1276-1002-1-ND" H 4400 -4000 50  0001 C CNN "SN-DK"
-F 5 "CL05B104KP5NNNC" H 4400 -4000 50  0001 C CNN "PN"
+F 5 "CL05C100JB5NNNC" H 0   0   50  0001 C CNN "PN"
 	1    8900 2950
 	-1   0    0    -1
@@
 F 2 "pkl_dipol:R_0402" V 1580 1400 50  0001 C CNN
 F 3 "~" H 1650 1400 50  0001 C CNN
+F 4 "Stackpole Electronics Inc" H 0   0   50  0001 C CNN "Mfg"
+F 5 "RMCF0402FT124K" H 0   0   50  0001 C CNN "PN"
 	1    1650 1400
 	1    0    0    1
@@
 F 2 "gkl_conn:SB02B-PASK-2" H 950 1100 50  0001 C CNN
 F 3 "~" H 950 1100 50  0001 C CNN
+F 4 "JST Sales America Inc." H 0   0   50  0001 C CNN "Mfg"
+F 5 "S02B-PASK-2(LF)(SN)" H 0   0   50  0001 C CNN "PN"
 	1    950  1100
 	1    0    0    -1
@@
 F 2 "pkl_dipol:R_0402" V 1580 1800 50  0001 C CNN
 F 3 "~" H 1650 1800 50  0001 C CNN
+F 4 "Stackpole Electronics Inc" H 0   0   50  0001 C CNN "Mfg"
+F 5 "RMCF0402FT124K" H 0   0   50  0001 C CNN "PN"
 	1    1650 1800
 	1    0    0    1
@@
 F 2 "pkl_dipol:R_0402" V 1580 2200 50  0001 C CNN
 F 3 "~" H 1650 2200 50  0001 C CNN
+F 4 "Stackpole Electronics Inc" H 0   0   50  0001 C CNN "Mfg"
+F 5 "RMCF0402FT124K" H 0   0   50  0001 C CNN "PN"
 	1    1650 2200
 	1    0    0    1
@@
 F 2 "pkl_dipol:R_0402" V 2830 1700 50  0001 C CNN
 F 3 "~" H 2900 1700 50  0001 C CNN
+F 4 "Stackpole Electronics Inc" H 0   0   50  0001 C CNN "Mfg"
+F 5 "RMCF0402FT510K" H 0   0   50  0001 C CNN "PN"
 	1    2900 1700
 	0    -1   1    0
@@
 F 2 "pkl_dipol:C_0805" H 5338 1550 50  0001 C CNN
 F 3 "" H 5300 1700 50  0001 C CNN
-F 4 "1276-1002-1-ND" H 800 -5250 50  0001 C CNN "SN-DK"
-F 5 "CL05B104KP5NNNC" H 800 -5250 50  0001 C CNN "PN"
+F 4 "CL21A106KAFN3NE" H 0   0   50  0001 C CNN "PN"
 	1    5300 1700
 	-1   0    0    -1
@@
 F 2 "pkl_dipol:C_0603" H 5688 1550 50  0001 C CNN
 F 3 "" H 5650 1700 50  0001 C CNN
-F 4 "1276-1002-1-ND" H 1150 -5250 50  0001 C CNN "SN-DK"
-F 5 "CL05B104KP5NNNC" H 1150 -5250 50  0001 C CNN "PN"
+F 4 "CL10B104KB8NNNC" H 0   0   50  0001 C CNN "PN"
 	1    5650 1700
 	-1   0    0    -1
@@
 F 2 "pkl_dipol:C_0805" H 7488 1550 50  0001 C CNN
 F 3 "" H 7450 1700 50  0001 C CNN
-F 4 "1276-1002-1-ND" H 2950 -5250 50  0001 C CNN "SN-DK"
-F 5 "CL05B104KP5NNNC" H 2950 -5250 50  0001 C CNN "PN"
+F 4 "CL21A106KAFN3NE" H 0   0   50  0001 C CNN "PN"
 	1    7450 1700
 	-1   0    0    -1
@@
 F 2 "pkl_dipol:C_0805" H 7788 1550 50  0001 C CNN
 F 3 "" H 7750 1700 50  0001 C CNN
-F 4 "1276-1002-1-ND" H 3250 -5250 50  0001 C CNN "SN-DK"
-F 5 "CL05B104KP5NNNC" H 3250 -5250 50  0001 C CNN "PN"
+F 4 "CL21A106KAFN3NE" H 0   0   50  0001 C CNN "PN"
 	1    7750 1700
 	-1   0    0    -1
@@
 F 2 "pkl_dipol:R_0402" V 8230 1150 50  0001 C CNN
 F 3 "~" H 8300 1150 50  0001 C CNN
+F 4 "Stackpole Electronics Inc" H 0   0   50  0001 C CNN "Mfg"
+F 5 "RMCF0402FT10K0" H 0   0   50  0001 C CNN "PN"
 	1    8300 1150
 	0    1    -1   0
@@
 F 2 "pkl_dipol:R_0402" V 8230 1300 50  0001 C CNN
 F 3 "~" H 8300 1300 50  0001 C CNN
+F 4 "Stackpole Electronics Inc" H 0   0   50  0001 C CNN "Mfg"
+F 5 "RMCF0402FT10K0" H 0   0   50  0001 C CNN "PN"
 	1    8300 1300
 	0    1    -1   0
