File: hardware/ButterStick_r0.3/SYZYGY_PORT1.sch (KiCad schematic (older format))
At the start: 2 parts, among them U3 ECP5U25

Commit message: hw.r0_3: Experiment with buses
Parts:
- removed U3: ECP5U25, gkl_housings_bga:caBGA_381_17x17, symbol gkl_lattice:ECP5U25-BG381
- R26: footprint pkl_dipol:R_0402 -> Resistor_SMD:R_0402_1005Metric
Other:
- note removed: "BANK3 - 1V8"
Changed lines of the file:
@@
 $Descr A4 11693 8268
 encoding utf-8
-Sheet 8 15
+Sheet 13 16
 Title "ButterStick"
 Date "2019-06-14"
@@
 $EndDescr
 Wire Wire Line
-	3650 2450 4600 2450
-Wire Wire Line
-	3650 2550 4600 2550
-Wire Wire Line
-	3650 2650 4600 2650
-Wire Wire Line
-	3650 2750 4600 2750
-Wire Wire Line
-	3650 2850 4100 2850
-Wire Wire Line
-	3650 2950 4100 2950
-Wire Wire Line
-	3650 3050 4100 3050
-Wire Wire Line
-	3650 3150 4100 3150
-Wire Wire Line
-	3650 3250 4300 3250
-Wire Wire Line
-	3650 3350 4300 3350
-Wire Wire Line
-	3650 3450 4100 3450
-Wire Wire Line
-	3650 3550 4100 3550
-Wire Wire Line
-	3650 3650 4300 3650
-Wire Wire Line
-	3650 3750 4300 3750
-Wire Wire Line
-	3650 3850 4100 3850
-Wire Wire Line
-	3650 3950 4100 3950
-Wire Wire Line
-	3650 4050 4300 4050
-Wire Wire Line
-	3650 4150 4300 4150
-Wire Wire Line
-	3650 4250 4100 4250
-Wire Wire Line
-	3650 4350 4100 4350
-Wire Wire Line
-	3650 4450 4300 4450
-Wire Wire Line
-	3650 4550 4300 4550
-Wire Wire Line
-	3650 4650 4100 4650
-Wire Wire Line
-	3650 4750 4100 4750
-Wire Wire Line
-	3650 4850 4300 4850
-Wire Wire Line
-	3650 4950 4300 4950
-Wire Wire Line
-	3650 5050 4300 5050
-Wire Wire Line
-	3650 5150 4300 5150
-Wire Wire Line
-	3650 5250 4300 5250
-Wire Wire Line
-	3650 5350 4300 5350
-Wire Wire Line
-	3650 5450 4300 5450
-Wire Wire Line
-	3650 5550 4300 5550
-Wire Wire Line
 	6500 2300 6050 2300
 Wire Wire Line
@@
 	8150 2600 8550 2600
 Wire Wire Line
-	8150 2800 8550 2800
-Wire Wire Line
-	8150 2900 8550 2900
-Wire Wire Line
-	8150 3100 8800 3100
-Wire Wire Line
 	8150 3200 8400 3200
 Wire Wire Line
 	8400 3200 8400 3500
-Text Notes 2500 2250 0    50   ~ 0
-BANK3 - 1V8
-Text Label 4100 2850 2    50   ~ 0
-S17
-Text Label 4100 2950 2    50   ~ 0
-S21
-Text Label 4100 3050 2    50   ~ 0
-S20
-Text Label 4100 3150 2    50   ~ 0
-S23
-Text Label 4100 3450 2    50   ~ 0
-S26
-Text Label 4100 3550 2    50   ~ 0
-S27
-Text Label 4100 3850 2    50   ~ 0
-S19
-Text Label 4100 3950 2    50   ~ 0
-S25
-Text Label 4100 4250 2    50   ~ 0
-S18
-Text Label 4100 4350 2    50   ~ 0
-S16
-Text Label 4100 4650 2    50   ~ 0
-S24
-Text Label 4100 4750 2    50   ~ 0
-S22
-Text Label 4300 3250 2    50   ~ 0
-D0_P
-Text Label 4300 3350 2    50   ~ 0
-D0_N
-Text Label 4300 3650 2    50   ~ 0
-D2_P
-Text Label 4300 3750 2    50   ~ 0
-D2_N
-Text Label 4300 4050 2    50   ~ 0
-D6_P
-Text Label 4300 4150 2    50   ~ 0
-D6_N
-Text Label 4300 4450 2    50   ~ 0
-D4_P
-Text Label 4300 4550 2    50   ~ 0
-D4_N
-Text Label 4300 4850 2    50   ~ 0
-D7_P
-Text Label 4300 4950 2    50   ~ 0
-D7_N
-Text Label 4300 5050 2    50   ~ 0
-D5_P
-Text Label 4300 5150 2    50   ~ 0
-D5_N
-Text Label 4300 5250 2    50   ~ 0
-D3_P
-Text Label 4300 5350 2    50   ~ 0
-D3_N
-Text Label 4300 5450 2    50   ~ 0
-D1_P
-Text Label 4300 5550 2    50   ~ 0
-D1_N
-Text Label 4600 2450 2    50   ~ 0
-C2P_CLK_P
-Text Label 4600 2550 2    50   ~ 0
-C2P_CLK_N
-Text Label 4600 2650 2    50   ~ 0
-P2C_CLK_P
-Text Label 4600 2750 2    50   ~ 0
-P2C_CLK_N
 Text Label 5850 5200 0    50   ~ 0
 P2C_CLK_P
@@
 Text HLabel 8550 2400 2    50   Input ~ 0
 EN
-Text HLabel 8550 2800 2    50   Input ~ 0
-pmicSCL
-Text HLabel 8550 2900 2    50   Input ~ 0
-pmicSDA
 $Comp
 L gkl_power:GND #PWR?
@@
 $EndComp
 $Comp
-L gkl_power:GND #PWR?
-U 1 1 5C996E43
-P 8800 3100
-AR Path="/5C80F1A0/5C996E43" Ref="#PWR?"  Part="1"
-AR Path="/5C80F19D/5C996E43" Ref="#PWR0215"  Part="1"
-F 0 "#PWR0215" H 8800 2850 50  0001 C CNN
-F 1 "GND" V 8804 3020 50  0000 R CNN
-F 2 "" H 8700 2750 50  0001 C CNN
-F 3 "" H 8800 3100 50  0001 C CNN
-	1    8800 3100
-	0    -1   -1   0
-$EndComp
-$Comp
 L Device:R R?
 U 1 1 5C996E36
@@
 F 0 "R26" H 8470 3696 50  0000 L CNN
 F 1 "84k5" H 8470 3605 50  0000 L CNN
-F 2 "pkl_dipol:R_0402" V 8330 3650 50  0001 C CNN
+F 2 "Resistor_SMD:R_0402_1005Metric" V 8330 3650 50  0001 C CNN
 F 3 "~" H 8400 3650 50  0001 C CNN
 F 4 "Stackpole Electronics Inc" H 0   0   50  0001 C CNN "Mfg"
@@
 	1    8400 3650
 	1    0    0    -1
-$EndComp
-$Comp
-L gkl_lattice:ECP5U25-BG381 U?
-U 4 1 5C810715
-P 3650 2450
-AR Path="/5AB8ACB7/5C810715" Ref="U?"  Part="4"
-AR Path="/5C80F19D/5C810715" Ref="U3"  Part="4"
-F 0 "U3" H 4600 2600 60  0000 L CNN
-F 1 "ECP5U25" H 3850 2600 60  0000 L CNN
-F 2 "gkl_housings_bga:caBGA_381_17x17" H 3650 2450 50  0001 C CNN
-F 3 "" H 3650 2450 50  0001 C CNN
-F 4 " 220-2052-ND " H -200 -1950 50  0001 C CNN "SN-DK"
-F 5 "LFE5U-45F-8BG381C" H -200 -1950 50  0001 C CNN "PN"
-F 6 "Lattice" H -200 -1950 50  0001 C CNN "Mfg"
-	4    3650 2450
-	-1   0    0    -1
 $EndComp
 $Sheet
@@
 F34 "SCL" I R 8150 2500 50
 F35 "SDA" I R 8150 2600 50
-F36 "PMIC_SCL" I R 8150 2800 50
-F37 "PMIC_SDA" I R 8150 2900 50
-F38 "PMIC_ADR0" I R 8150 3100 50
-F39 "VCCIO" I R 8150 2300 50
-F40 "R_GA" I R 8150 3200 50
-F41 "PMIC_EN" I R 8150 2400 50
+F36 "VCCIO" I R 8150 2300 50
+F37 "R_GA" I R 8150 3200 50
+F38 "PMIC_EN" I R 8150 2400 50
 $EndSheet
 $EndSCHEMATC

Commit message: hw.r0_3: cleanup and additions
Parts:
- removed R26: 84k5, Resistor_SMD:R_0402_1005Metric, symbol Device:R
Changed lines of the file:
@@
 $Descr A4 11693 8268
 encoding utf-8
-Sheet 13 16
+Sheet 5 20
 Title "ButterStick"
 Date "2019-06-14"
@@
 	1    0    0    -1
 $EndComp
-$Comp
-L Device:R R?
-U 1 1 5C996E36
-P 8400 3650
-AR Path="/5C80F1A0/5C996E36" Ref="R?"  Part="1"
-AR Path="/5C80F19D/5C996E36" Ref="R26"  Part="1"
-F 0 "R26" H 8470 3696 50  0000 L CNN
-F 1 "84k5" H 8470 3605 50  0000 L CNN
-F 2 "Resistor_SMD:R_0402_1005Metric" V 8330 3650 50  0001 C CNN
-F 3 "~" H 8400 3650 50  0001 C CNN
-F 4 "Stackpole Electronics Inc" H 0   0   50  0001 C CNN "Mfg"
-F 5 "RMCF0402FT84K5" H 0   0   50  0001 C CNN "PN"
-F 6 "1%" H 0   0   50  0001 C CNN "Tol"
-	1    8400 3650
-	1    0    0    -1
-$EndComp
