File: hardware/ButterStick_r0.3/SYZYGY_PORT2.sch (KiCad schematic (older format))
At the start: 2 parts, among them U3 ECP5U25

Commit message: hw.r0_3: Experiment with buses
Parts:
- R28: footprint pkl_dipol:R_0402 -> Resistor_SMD:R_0402_1005Metric
Changed lines of the file:
@@
 $Descr A4 11693 8268
 encoding utf-8
-Sheet 10 15
+Sheet 9 16
 Title "ButterStick"
 Date "2019-06-14"
@@
 F 0 "R28" H 9020 3746 50  0000 L CNN
 F 1 "49k9" H 9020 3655 50  0000 L CNN
-F 2 "pkl_dipol:R_0402" V 8880 3700 50  0001 C CNN
+F 2 "Resistor_SMD:R_0402_1005Metric" V 8880 3700 50  0001 C CNN
 F 3 "~" H 8950 3700 50  0001 C CNN
 F 4 "Stackpole Electronics Inc" H 0   0   50  0001 C CNN "Mfg"

Commit message: hw.r0_3: cleanup and additions
Parts:
- removed R28: 49k9, Resistor_SMD:R_0402_1005Metric, symbol Device:R
Changed lines of the file:
@@
 $Descr A4 11693 8268
 encoding utf-8
-Sheet 9 16
+Sheet 9 20
 Title "ButterStick"
 Date "2019-06-14"
@@
 	1    0    0    -1
 $EndComp
-$Comp
-L Device:R R28
-U 1 1 5C986FFC
-P 8950 3700
-F 0 "R28" H 9020 3746 50  0000 L CNN
-F 1 "49k9" H 9020 3655 50  0000 L CNN
-F 2 "Resistor_SMD:R_0402_1005Metric" V 8880 3700 50  0001 C CNN
-F 3 "~" H 8950 3700 50  0001 C CNN
-F 4 "Stackpole Electronics Inc" H 0   0   50  0001 C CNN "Mfg"
-F 5 "RMCF0402FT49K9" H 0   0   50  0001 C CNN "PN"
-F 6 "1%" H 0   0   50  0001 C CNN "Tol"
-	1    8950 3700
-	1    0    0    -1
-$EndComp
