File: hardware/ButterStick_r0.3/FPGA-SYZGY1.sch (KiCad schematic (older format))
At the start: 1 part, among them U2 ECP5UM5G_85_CABGA381

Commit message: hw.r0_3: Start pin assignments for DDR3
Parts:
- U2: symbol ECP5UM5G-85Pinout:ECP5UM5G_85_CABGA381 -> gkl_lattice:ECP5UM5G_85_CABGA381
Connections:
- net D0_N: now reaches U2.F1 (PL47B/PCLKC6_1/LDQ53)
- net D1_N: now reaches U2.G1 (PL47D/PCLKC6_0/LDQ53)
- net D5_P: now reaches U2.H1 (PL53C/LDQ53)
- net D1_P: now reaches U2.H2 (PL47C/PCLKT6_0/LDQ53)
- net D4_N: now reaches U2.J1 (PL53B/LDQSN53)
- net D3_P: now reaches U2.J3 (PL50C/GR_PCLK6_1/LDQ53)
- net D2_P: now reaches U2.J4 (PL50A/GR_PCLK6_0/LDQ53)
- net D2_N: now reaches U2.J5 (PL50B/LDQ53)
- net D5_N: now reaches U2.K1 (PL53D/LDQ53)
- net D4_P: now reaches U2.K2 (PL53A/LDQS53)
- net D3_N: now reaches U2.K3 (PL50D/LDQ53)
- net D6_P: now reaches U2.K4 (PL56A/LDQ53)
- net D6_N: now reaches U2.K5 (PL56B/VREF1_6/LDQ53)
- net S27: now reaches U2.L1 (PL89C/LDQ89)
- net S24: now reaches U2.L2 (PL86D/LDQ89)
- net S23: now reaches U2.L3 (PL86C/LDQ89)
- net D7_P: now reaches U2.L4 (PL56C/LDQ53)
- net D7_N: now reaches U2.L5 (PL56D/LDQ53)
- net VIO1: now reaches U2.L6 (VCCIO6[3]), U2.L7 (VCCIO6[3]), U2.M6 (VCCIO6[3])
- net S26: now reaches U2.M1 (PL89B/LDQSN89)
- net S22: now reaches U2.M3 (PL86B/LDQ89)
- net S17: now reaches U2.M4 (PL83A/LDQ89)
- net S16: now reaches U2.M5 (PL77A/LDQS77)
- net C2P_CLK_P: now reaches U2.N1 (PL89D/LDQ89)
- net S25: now reaches U2.N2 (PL89A/LDQS89)
- net S21: now reaches U2.N3 (PL86A/LDQ89)
- net S19: now reaches U2.N4 (PL83C/LDQ89)
- net S18: now reaches U2.N5 (PL83B/LDQ89)
- net C2P_CLK_N: now reaches U2.P1 (PL92A/LDQ89)
- net P2C_CLK_P: now reaches U2.P2 (PL92B/LDQ89)
- net P2C_CLK_N: now reaches U2.P3 (PL92C/LLC_GPLL0T_IN/LDQ89)
- net S20: now reaches U2.P5 (PL83D/LDQ89)
- net S0_D0P renamed D0_P
Changed lines of the file:
@@
 $Descr A4 11693 8268
 encoding utf-8
-Sheet 10 18
+Sheet 11 20
 Title ""
 Date ""
@@
 $EndDescr
 Entry Wire Line
+	4100 2050 4200 1950
+Entry Wire Line
 	4200 2900 4300 2800
+Entry Wire Line
+	4200 3000 4300 2900
+Entry Wire Line
+	4200 3100 4300 3000
+Entry Wire Line
+	4200 3200 4300 3100
+Entry Wire Line
+	4200 3300 4300 3200
+Entry Wire Line
+	4200 3400 4300 3300
+Entry Wire Line
+	4200 3500 4300 3400
+Entry Wire Line
+	4200 3600 4300 3500
+Entry Wire Line
+	4200 3700 4300 3600
+Entry Wire Line
+	4200 3800 4300 3700
+Entry Wire Line
+	4200 3900 4300 3800
+Entry Wire Line
+	4200 4000 4300 3900
+Entry Wire Line
+	4200 4100 4300 4000
+Entry Wire Line
+	4200 4200 4300 4100
+Entry Wire Line
+	4200 4300 4300 4200
+Entry Wire Line
+	4200 4400 4300 4300
+Entry Wire Line
+	4200 4500 4300 4400
+Entry Wire Line
+	4200 4600 4300 4500
+Entry Wire Line
+	4200 4700 4300 4600
+Entry Wire Line
+	4200 4800 4300 4700
+Entry Wire Line
+	4200 4900 4300 4800
+Entry Wire Line
+	4200 5000 4300 4900
+Entry Wire Line
+	4200 5100 4300 5000
+Entry Wire Line
+	4200 5200 4300 5100
+Entry Wire Line
+	4200 5300 4300 5200
+Entry Wire Line
+	4200 5400 4300 5300
+Entry Wire Line
+	4200 5500 4300 5400
+Entry Wire Line
+	4200 5600 4300 5500
+Entry Wire Line
+	4200 5700 4300 5600
+Entry Wire Line
+	4200 5800 4300 5700
+Entry Wire Line
+	4200 5900 4300 5800
+Entry Wire Line
+	4200 6000 4300 5900
+Wire Wire Line
+	4200 1950 6200 1950
 Wire Wire Line
 	4300 2800 4700 2800
+Wire Wire Line
+	4300 2900 4700 2900
+Wire Wire Line
+	4300 3000 4700 3000
+Wire Wire Line
+	4300 3100 4700 3100
+Wire Wire Line
+	4300 3200 4700 3200
+Wire Wire Line
+	4300 3300 4700 3300
+Wire Wire Line
+	4300 3400 4700 3400
+Wire Wire Line
+	4300 3500 4700 3500
+Wire Wire Line
+	4300 3600 4700 3600
+Wire Wire Line
+	4300 3700 4700 3700
+Wire Wire Line
+	4300 3800 4700 3800
+Wire Wire Line
+	4300 3900 4700 3900
+Wire Wire Line
+	4300 4000 4700 4000
+Wire Wire Line
+	4300 4100 4700 4100
+Wire Wire Line
+	4300 4200 4700 4200
+Wire Wire Line
+	4300 4300 4700 4300
+Wire Wire Line
+	4300 4400 4700 4400
+Wire Wire Line
+	4300 4500 4700 4500
+Wire Wire Line
+	4300 4600 4700 4600
+Wire Wire Line
+	4300 4700 4700 4700
+Wire Wire Line
+	4300 4800 4700 4800
+Wire Wire Line
+	4300 4900 4700 4900
+Wire Wire Line
+	4300 5000 4700 5000
+Wire Wire Line
+	4300 5100 4700 5100
+Wire Wire Line
+	4300 5200 4700 5200
+Wire Wire Line
+	4300 5300 4700 5300
+Wire Wire Line
+	4300 5400 4700 5400
+Wire Wire Line
+	4300 5500 4700 5500
+Wire Wire Line
+	4300 5600 4700 5600
+Wire Wire Line
+	4300 5700 4700 5700
+Wire Wire Line
+	4300 5800 4700 5800
+Wire Wire Line
+	4300 5900 4700 5900
+Wire Wire Line
+	6200 1950 6200 2500
 Wire Bus Line
 	1300 2050 4200 2050
 Wire Bus Line
-	4200 2050 4200 6000
-Text Notes 6250 2600 2    50   ~ 0
+	4200 2050 4200 2900
+Wire Bus Line
+	4200 2900 4200 3100
+Wire Bus Line
+	4200 3100 4200 3300
+Wire Bus Line
+	4200 3300 4200 3500
+Wire Bus Line
+	4200 3500 4200 3600
+Wire Bus Line
+	4200 3600 4200 3800
+Wire Bus Line
+	4200 3800 4200 4000
+Wire Bus Line
+	4200 4000 4200 4100
+Wire Bus Line
+	4200 4100 4200 4300
+Wire Bus Line
+	4200 4300 4200 4500
+Wire Bus Line
+	4200 4500 4200 4700
+Wire Bus Line
+	4200 4700 4200 4800
+Wire Bus Line
+	4200 4800 4200 5000
+Wire Bus Line
+	4200 5000 4200 5100
+Wire Bus Line
+	4200 5100 4200 5300
+Wire Bus Line
+	4200 5300 4200 5500
+Wire Bus Line
+	4200 5500 4200 5700
+Wire Bus Line
+	4200 5700 4200 5900
+Wire Bus Line
+	4200 5900 4200 6000
+Text Notes 5850 2500 2    50   ~ 0
 PIC Differential Mappings\n - PIOA/B : Transmit/Receive\n - PIOC/D : Receive
+Text Label 4300 1950 0    50   ~ 0
+VIO1
 Text Label 4300 2800 0    50   ~ 0
-S0_D0P
+D0_P
+Text Label 4300 2900 0    50   ~ 0
+D0_N
+Text Label 4300 3000 0    50   ~ 0
+D1_P
+Text Label 4300 3100 0    50   ~ 0
+D1_N
+Text Label 4300 3200 0    50   ~ 0
+D2_P
+Text Label 4300 3300 0    50   ~ 0
+D2_N
+Text Label 4300 3400 0    50   ~ 0
+D3_P
+Text Label 4300 3500 0    50   ~ 0
+D3_N
+Text Label 4300 3600 0    50   ~ 0
+D4_P
+Text Label 4300 3700 0    50   ~ 0
+D4_N
+Text Label 4300 3800 0    50   ~ 0
+D5_P
+Text Label 4300 3900 0    50   ~ 0
+D5_N
+Text Label 4300 4000 0    50   ~ 0
+D6_P
+Text Label 4300 4100 0    50   ~ 0
+D6_N
+Text Label 4300 4200 0    50   ~ 0
+D7_P
+Text Label 4300 4300 0    50   ~ 0
+D7_N
+Text Label 4300 4400 0    50   ~ 0
+S16
+Text Label 4300 4500 0    50   ~ 0
+S17
+Text Label 4300 4600 0    50   ~ 0
+S18
+Text Label 4300 4700 0    50   ~ 0
+S19
+Text Label 4300 4800 0    50   ~ 0
+S20
+Text Label 4300 4900 0    50   ~ 0
+S21
+Text Label 4300 5000 0    50   ~ 0
+S22
+Text Label 4300 5100 0    50   ~ 0
+S23
+Text Label 4300 5200 0    50   ~ 0
+S24
+Text Label 4300 5300 0    50   ~ 0
+S25
+Text Label 4300 5400 0    50   ~ 0
+S26
+Text Label 4300 5500 0    50   ~ 0
+S27
+Text Label 4300 5600 0    50   ~ 0
+C2P_CLK_P
+Text Label 4300 5700 0    50   ~ 0
+C2P_CLK_N
+Text Label 4300 5800 0    50   ~ 0
+P2C_CLK_P
+Text Label 4300 5900 0    50   ~ 0
+P2C_CLK_N
 Text HLabel 1300 2050 0    50   Input ~ 0
 {SYZYGY_STD}
 $Comp
-L ECP5UM5G-85Pinout:ECP5UM5G_85_CABGA381 U2
+L gkl_lattice:ECP5UM5G_85_CABGA381 U2
 U 6 1 5E95CD57
 P 4700 2800
