File: hardware/ButterStick_r0.3/SyzygyStandard.sch (KiCad schematic (older format))
At the start: 14 parts, among them J1 SYZYGY-STD, U2 DAC081C081CIMK, U7 TPS73101DBV

Commit message: hw.r0_3: Experiment with buses
Parts:
- removed C1: 4.7uF, pkl_dipol:C_0603, symbol Device:C
- removed R1: 42k2, pkl_dipol:C_0402, symbol Device:R
- removed TP10: TestPoint_Flag, gkl_conn:TestPoint_Pad_D1.0mm, symbol Connector:TestPoint_Flag
- removed U2: DAC081C081CIMK, Package_TO_SOT_SMD:SOT-23-6, symbol Analog_DAC:DAC081C081CIMK
- removed U7: TPS73101DBV, Package_TO_SOT_SMD:SOT-23-5, symbol Regulator_Linear:TPS73101DBV
- added C43: 1uF, Capacitor_SMD:C_0402_1005Metric, symbol Device:C
- added C46, C47: 4.7uF, Capacitor_SMD:C_0603_1608Metric, symbol Device:C
- added Q1: PMBT3904MB, Package_TO_SOT_SMD:SOT-883, symbol gkl_misc:PMBT3904MB
- added R18: 10K, Resistor_SMD:R_0402_1005Metric, symbol Device:R
- added U2: TLV6001DCK, Package_TO_SOT_SMD:SOT-353_SC-70-5, symbol Amplifier_Operational:TLV6001DCK
- C2, C95: footprint pkl_dipol:C_0402 -> Capacitor_SMD:C_0402_1005Metric
- C24: footprint pkl_dipol:C_0603 -> Capacitor_SMD:C_0603_1608Metric
- R2: value 33K -> 10K; footprint pkl_dipol:C_0402 -> Resistor_SMD:R_0402_1005Metric; PN RNCF0402DTE33K0 -> (none); Tol 0.5% -> 1%
- R29: footprint pkl_dipol:R_0402 -> Resistor_SMD:R_0402_1005Metric
- R5: value 24k9 -> 10K; footprint pkl_dipol:C_0402 -> Resistor_SMD:R_0402_1005Metric; PN RNCF0402DTE24K9 -> (none); Tol 0.5% -> 1%
- R63: footprint pkl_dipol:C_0402 -> Resistor_SMD:R_0402_1005Metric
Connections:
- net labels added: VCCIO_PDM
- net labels removed: PMIC_ADR0, PMIC_EN, PMIC_SCL, PMIC_SDA
- wire segments 76 -> 83
Other:
- note added: "Max power dissipation\n400mW"
- moved on the sheet: C2, C24, C95, J1, R2, R31, R5, R63, TP13

Commit message: hw.r0_3: cleanup and additions
Parts:
- removed R29: 0R, Resistor_SMD:R_0402_1005Metric, symbol Device:R
- added JP2: Jumper_NC, Jumper:SolderJumper-2_P1.3mm_Bridged2Bar_RoundedPad1.0x1.5mm, symbol Device:Jumper_NC_Small
- TP11: value TestPoint_Flag -> VCCIO_TP
Connections:
- net VOUT: now also JP2.1
- net C2P_CLKn renamed C2P_CLKN
- net C2P_CLKp renamed C2P_CLKP
- net D0n renamed S2_D0N
- net D0p renamed S0_D0P
- net D1n renamed S3_D1N
- net D1p renamed S1_D1P
- net D2n renamed S6_D2N
- net D2p renamed S4_D2P
- net D3n renamed S7_D3N
- net D3p renamed S5_D3P
- net D4n renamed S10_D4N
- net D4p renamed S8_D4P
- net D5n renamed S11_D5N
- net D5p renamed S9_D5P
- net D6n renamed S14_D6N
- net D6p renamed S12_D6P
- net D7n renamed S15_D7N
- net D7p renamed S13_D7P
- net P2C_CLKn renamed P2C_CLKN
- net P2C_CLKp renamed P2C_CLKP
- net VCCIO renamed VIO1
- net VIO1: now also JP2.2
Other:
- moved on the sheet: C2, C43, R18, R63, TP13

Commit message: hw.r0_3: Start pin assignments for DDR3
Parts:
- JP2: footprint Jumper:SolderJumper-2_P1.3mm_Bridged2Bar_RoundedPad1.0x1.5mm -> NetTie:NetTie-2_SMD_Pad0.5mm
Connections:
- net C2P_CLKN renamed C2P_CLK_N
- net C2P_CLKP renamed C2P_CLK_P
- net P2C_CLKN renamed P2C_CLK_N
- net P2C_CLKP renamed P2C_CLK_P
- net S0_D0P renamed D0_P
- net S10_D4N renamed D4_N
- net S11_D5N renamed D5_N
- net S12_D6P renamed D6_P
- net S13_D7P renamed D7_P
- net S14_D6N renamed D6_N
- net S15_D7N renamed D7_N
- net S1_D1P renamed D1_P
- net S2_D0N renamed D0_N
- net S3_D1N renamed D1_N
- net S4_D2P renamed D2_P
- net S5_D3P renamed D3_P
- net S6_D2N renamed D2_N
- net S7_D3N renamed D3_N
- net S8_D4P renamed D4_P
- net S9_D5P renamed D5_P
Changed lines of the file:
@@
 $Descr A4 11693 8268
 encoding utf-8
-Sheet 14 18
+Sheet 18 20
 Title "ButterStick"
 Date "2019-06-14"
@@
 	6350 6050 6500 6050
 Wire Bus Line
-	6500 4000 6500 4100
-Wire Bus Line
-	6500 4100 6500 4300
-Wire Bus Line
-	6500 4300 6500 4500
-Wire Bus Line
-	6500 4500 6500 4700
+	6500 4000 6500 4200
+Wire Bus Line
+	6500 4200 6500 4400
+Wire Bus Line
+	6500 4400 6500 4600
+Wire Bus Line
+	6500 4600 6500 4700
 Wire Bus Line
 	6500 4700 6500 4900
@@
 	9000 4000 9000 4200
 Wire Bus Line
-	9000 4200 9000 4300
-Wire Bus Line
-	9000 4300 9000 4500
+	9000 4200 9000 4400
+Wire Bus Line
+	9000 4400 9000 4500
 Wire Bus Line
 	9000 4500 9000 4700
 Wire Bus Line
-	9000 4700 9000 4900
-Wire Bus Line
-	9000 4900 9000 5100
-Wire Bus Line
-	9000 5100 9000 5200
-Wire Bus Line
-	9000 5200 9000 5400
+	9000 4700 9000 4800
+Wire Bus Line
+	9000 4800 9000 5000
+Wire Bus Line
+	9000 5000 9000 5100
+Wire Bus Line
+	9000 5100 9000 5300
+Wire Bus Line
+	9000 5300 9000 5400
 Wire Bus Line
 	9000 5400 9000 6050
@@
 SDA
 Text Label 6600 3900 0    50   ~ 0
-S0_D0P
+D0_P
 Text Label 6600 4000 0    50   ~ 0
-S2_D0N
+D0_N
 Text Label 6600 4100 0    50   ~ 0
-S4_D2P
+D2_P
 Text Label 6600 4200 0    50   ~ 0
-S6_D2N
+D2_N
 Text Label 6600 4300 0    50   ~ 0
-S8_D4P
+D4_P
 Text Label 6600 4400 0    50   ~ 0
-S10_D4N
+D4_N
 Text Label 6600 4500 0    50   ~ 0
-S12_D6P
+D6_P
 Text Label 6600 4600 0    50   ~ 0
-S14_D6N
+D6_N
 Text Label 6600 4700 0    50   ~ 0
 S16
@@
 S26
 Text Label 6600 5300 0    50   ~ 0
-P2C_CLKP
+P2C_CLK_P
 Text Label 6600 5400 0    50   ~ 0
-P2C_CLKN
+P2C_CLK_N
 Text Label 6700 5700 0    50   ~ 0
 VIO1
@@
 R_GA
 Text Label 8900 3900 2    50   ~ 0
-S1_D1P
+D1_P
 Text Label 8900 4000 2    50   ~ 0
-S3_D1N
+D1_N
 Text Label 8900 4100 2    50   ~ 0
-S5_D3P
+D3_P
 Text Label 8900 4200 2    50   ~ 0
-S7_D3N
+D3_N
 Text Label 8900 4300 2    50   ~ 0
-S9_D5P
+D5_P
 Text Label 8900 4400 2    50   ~ 0
-S11_D5N
+D5_N
 Text Label 8900 4500 2    50   ~ 0
-S13_D7P
+D7_P
 Text Label 8900 4600 2    50   ~ 0
-S15_D7N
+D7_N
 Text Label 8900 4700 2    50   ~ 0
 S17
@@
 S27
 Text Label 8900 5300 2    50   ~ 0
-C2P_CLKP
+C2P_CLK_P
 Text Label 8900 5400 2    50   ~ 0
-C2P_CLKN
+C2P_CLK_N
 Text HLabel 1400 2150 0    50   Input ~ 0
 VCCIO_PDM
@@
 AR Path="/5E9F0D55/5E93E49A" Ref="JP?"  Part="1"
 AR Path="/5E9F0D54/5E93E49A" Ref="JP?"  Part="1"
-F 0 "JP4" H 5750 1970 50  0000 C CNN
+F 0 "JP5" H 5750 1970 50  0000 C CNN
 F 1 "Jumper_NC" H 5750 1970 50  0001 C CNN
-F 2 "Jumper:SolderJumper-2_P1.3mm_Bridged2Bar_RoundedPad1.0x1.5mm" H 5750 1850 50  0001 C CNN
+F 2 "NetTie:NetTie-2_SMD_Pad0.5mm" H 5750 1850 50  0001 C CNN
 F 3 "~" H 5750 1850 50  0001 C CNN
 F 4 "DNP" H 5750 1850 50  0001 C CNN "PN"
@@
 AR Path="/5E9F0D55/5E95D8BF" Ref="R?"  Part="1"
 AR Path="/5E9F0D54/5E95D8BF" Ref="R?"  Part="1"
-F 0 "R7" V 1444 2150 50  0000 C CNN
+F 0 "R11" V 1444 2150 50  0000 C CNN
 F 1 "10K" V 1535 2150 50  0000 C CNN
 F 2 "Resistor_SMD:R_0402_1005Metric" V 1580 2150 50  0001 C CNN
@@
 AR Path="/5E9F0D55/5D15D762" Ref="R?"  Part="1"
 AR Path="/5E9F0D54/5D15D762" Ref="R?"  Part="1"
-F 0 "R8" H 1930 2454 50  0000 R CNN
+F 0 "R12" H 1930 2454 50  0000 R CNN
 F 1 "10K" H 1930 2545 50  0000 R CNN
 F 2 "Resistor_SMD:R_0402_1005Metric" V 1930 2500 50  0001 C CNN
@@
 AR Path="/5E9F0D55/5C939F38" Ref="R?"  Part="1"
 AR Path="/5E9F0D54/5C939F38" Ref="R?"  Part="1"
-F 0 "R9" H 4480 2105 50  0000 R CNN
+F 0 "R13" H 4480 2105 50  0000 R CNN
 F 1 "10K" H 4480 2195 50  0000 R CNN
 F 2 "Resistor_SMD:R_0402_1005Metric" V 4480 2150 50  0001 C CNN
@@
 AR Path="/5E9F0D55/5C939F3F" Ref="R?"  Part="1"
 AR Path="/5E9F0D54/5C939F3F" Ref="R?"  Part="1"
-F 0 "R10" H 4480 2605 50  0000 R CNN
+F 0 "R14" H 4480 2605 50  0000 R CNN
 F 1 "10K" H 4480 2695 50  0000 R CNN
 F 2 "Resistor_SMD:R_0402_1005Metric" V 4480 2650 50  0001 C CNN
@@
 AR Path="/5E9F0D55/5D166E9F" Ref="TP?"  Part="1"
 AR Path="/5E9F0D54/5D166E9F" Ref="TP?"  Part="1"
-F 0 "TP8" H 6610 1944 50  0000 L CNN
+F 0 "TP10" H 6610 1944 50  0000 L CNN
 F 1 "VCCIO_TP" H 6610 1853 50  0000 L CNN
 F 2 "gkl_conn:TestPoint_Pad_D1.0mm" H 6550 1850 50  0001 C CNN
@@
 AR Path="/5E9F0D55/5E95E788" Ref="C?"  Part="1"
 AR Path="/5E9F0D54/5E95E788" Ref="C?"  Part="1"
-F 0 "C74" H 2315 2545 50  0000 L CNN
+F 0 "C106" H 2315 2545 50  0000 L CNN
 F 1 "1uF" H 2315 2455 50  0000 L CNN
 F 2 "Capacitor_SMD:C_0402_1005Metric" H 2238 2350 50  0001 C CNN
@@
 AR Path="/5E9F0D55/5C939F1D" Ref="C?"  Part="1"
 AR Path="/5E9F0D54/5C939F1D" Ref="C?"  Part="1"
-F 0 "C101" H 3165 2445 50  0000 L CNN
+F 0 "C107" H 3165 2445 50  0000 L CNN
 F 1 "100nF" H 3165 2355 50  0000 L CNN
 F 2 "Capacitor_SMD:C_0402_1005Metric" H 3088 2250 50  0001 C CNN
@@
 AR Path="/5E9F0D55/5C939F46" Ref="C?"  Part="1"
 AR Path="/5E9F0D54/5C939F46" Ref="C?"  Part="1"
-F 0 "C102" H 4985 2445 50  0000 R CNN
+F 0 "C108" H 4985 2445 50  0000 R CNN
 F 1 "4.7uF" H 4985 2355 50  0000 R CNN
 F 2 "Capacitor_SMD:C_0603_1608Metric" H 5138 2250 50  0001 C CNN
@@
 AR Path="/5E9F0D55/5CF397B4" Ref="C?"  Part="1"
 AR Path="/5E9F0D54/5CF397B4" Ref="C?"  Part="1"
-F 0 "C103" H 5235 2445 50  0000 R CNN
+F 0 "C109" H 5235 2445 50  0000 R CNN
 F 1 "100nF" H 5235 2355 50  0000 R CNN
 F 2 "Capacitor_SMD:C_0402_1005Metric" H 5388 2250 50  0001 C CNN
@@
 AR Path="/5E9F0D55/5E9CC6DF" Ref="C?"  Part="1"
 AR Path="/5E9F0D54/5E9CC6DF" Ref="C?"  Part="1"
-F 0 "C104" H 7535 2845 50  0000 R CNN
+F 0 "C110" H 7535 2845 50  0000 R CNN
 F 1 "4.7uF" H 7535 2755 50  0000 R CNN
 F 2 "Capacitor_SMD:C_0603_1608Metric" H 7688 2650 50  0001 C CNN
@@
 AR Path="/5E9F0D55/5E9D4294" Ref="C?"  Part="1"
 AR Path="/5E9F0D54/5E9D4294" Ref="C?"  Part="1"
-F 0 "C105" H 7785 2845 50  0000 R CNN
+F 0 "C111" H 7785 2845 50  0000 R CNN
 F 1 "4.7uF" H 7785 2755 50  0000 R CNN
 F 2 "Capacitor_SMD:C_0603_1608Metric" H 7938 2650 50  0001 C CNN
@@
 AR Path="/5E9F0D55/5E94FAE6" Ref="Q?"  Part="1"
 AR Path="/5E9F0D54/5E94FAE6" Ref="Q?"  Part="1"
-F 0 "Q4" V 4427 1950 50  0000 C CNN
+F 0 "Q5" V 4427 1950 50  0000 C CNN
 F 1 "PMBT3904MB" V 4336 1950 50  0000 C CNN
 F 2 "Package_TO_SOT_SMD:SOT-883" H 4300 2050 50  0001 C CNN
@@
 AR Path="/5E9F0D55/5E93FD25" Ref="U?"  Part="1"
 AR Path="/5E9F0D54/5E93FD25" Ref="U?"  Part="1"
-F 0 "U10" H 3800 2050 50  0000 L CNN
+F 0 "U12" H 3800 2050 50  0000 L CNN
 F 1 "TLV6001DCK" H 3800 2150 50  0000 L CNN
 F 2 "Package_TO_SOT_SMD:SOT-353_SC-70-5" H 3800 2250 50  0001 C CNN
@@
 AR Path="/5E9F0D55/5C813052" Ref="J?"  Part="1"
 AR Path="/5E9F0D54/5C813052" Ref="J?"  Part="1"
-F 0 "J7" H 7750 5669 50  0000 C CNN
+F 0 "J9" H 7750 5669 50  0000 C CNN
 F 1 "SYZYGY-STD" H 7750 5578 50  0000 C CNN
 F 2 "gkl_conn:SYZYGY_standard_carrier" H 7750 5550 50  0001 C CNN
