File: hardware/ButterStick_r0.3/fileFPGA.sch (KiCad schematic (older format))
At the start: 18 parts, among them U3 ECP5U25, X1 ASDMB

Commit message: hw.r0_3: Experiment with buses
Parts:
- C100, C80, C81, C82, C83, C84, C85, C86, C87, C88, C89, C90, C91: footprint pkl_dipol:C_0402 -> Capacitor_SMD:C_0402_1005Metric
- R4, R47, R66: footprint pkl_dipol:R_0402 -> Resistor_SMD:R_0402_1005Metric
Changed lines of the file:
@@
 $Descr A4 11693 8268
 encoding utf-8
-Sheet 4 15
+Sheet 4 16
 Title "ButterStick"
 Date "2019-06-14"
@@
 F 0 "R66" V 2743 7100 50  0000 C CNN
 F 1 "20R" V 2834 7100 50  0000 C CNN
-F 2 "pkl_dipol:R_0402" V 2880 7100 50  0001 C CNN
+F 2 "Resistor_SMD:R_0402_1005Metric" V 2880 7100 50  0001 C CNN
 F 3 "~" H 2950 7100 50  0001 C CNN
 F 4 "Stackpole Electronics Inc" H 0   0   50  0001 C CNN "Mfg"
@@
 F 0 "R47" V 5057 1700 50  0000 C CNN
 F 1 "20R" V 4966 1700 50  0000 C CNN
-F 2 "pkl_dipol:R_0402" V 4780 1700 50  0001 C CNN
+F 2 "Resistor_SMD:R_0402_1005Metric" V 4780 1700 50  0001 C CNN
 F 3 "~" H 4850 1700 50  0001 C CNN
 F 4 "Stackpole Electronics Inc" H 0   0   50  0001 C CNN "Mfg"
@@
 F 0 "R4" H 9120 3396 50  0000 L CNN
 F 1 "4k7" H 9120 3305 50  0000 L CNN
-F 2 "pkl_dipol:R_0402" V 8980 3350 50  0001 C CNN
+F 2 "Resistor_SMD:R_0402_1005Metric" V 8980 3350 50  0001 C CNN
 F 3 "" H 9050 3350 50  0001 C CNN
 F 4 "P10KDECT-ND" H -1200 800 50  0001 C CNN "SN-DK"
@@
 F 0 "C80" H 4000 6250 50  0000 L CNN
 F 1 "100nF" H 4000 6050 50  0000 L CNN
-F 2 "pkl_dipol:C_0402" H 3988 6000 50  0001 C CNN
+F 2 "Capacitor_SMD:C_0402_1005Metric" H 3988 6000 50  0001 C CNN
 F 3 "" H 3950 6150 50  0001 C CNN
 F 4 "1276-1002-1-ND" H -1950 -800 50  0001 C CNN "SN-DK"
@@
 F 0 "C81" H 4000 7000 50  0000 L CNN
 F 1 "100nF" H 4000 6800 50  0000 L CNN
-F 2 "pkl_dipol:C_0402" H 3988 6750 50  0001 C CNN
+F 2 "Capacitor_SMD:C_0402_1005Metric" H 3988 6750 50  0001 C CNN
 F 3 "" H 3950 6900 50  0001 C CNN
 F 4 "1276-1002-1-ND" H -1950 -50 50  0001 C CNN "SN-DK"
@@
 F 0 "C82" H 4400 6250 50  0000 L CNN
 F 1 "10nF" H 4400 6050 50  0000 L CNN
-F 2 "pkl_dipol:C_0402" H 4388 6000 50  0001 C CNN
+F 2 "Capacitor_SMD:C_0402_1005Metric" H 4388 6000 50  0001 C CNN
 F 3 "" H 4350 6150 50  0001 C CNN
 F 4 "1276-1002-1-ND" H -1550 -800 50  0001 C CNN "SN-DK"
@@
 F 0 "C83" H 4400 7000 50  0000 L CNN
 F 1 "10nF" H 4400 6800 50  0000 L CNN
-F 2 "pkl_dipol:C_0402" H 4388 6750 50  0001 C CNN
+F 2 "Capacitor_SMD:C_0402_1005Metric" H 4388 6750 50  0001 C CNN
 F 3 "" H 4350 6900 50  0001 C CNN
 F 4 "1276-1002-1-ND" H -1550 -50 50  0001 C CNN "SN-DK"
@@
 F 0 "C84" H 4900 6250 50  0000 L CNN
 F 1 "100nF" H 4900 6050 50  0000 L CNN
-F 2 "pkl_dipol:C_0402" H 4888 6000 50  0001 C CNN
+F 2 "Capacitor_SMD:C_0402_1005Metric" H 4888 6000 50  0001 C CNN
 F 3 "" H 4850 6150 50  0001 C CNN
 F 4 "1276-1002-1-ND" H -1050 -800 50  0001 C CNN "SN-DK"
@@
 F 0 "C85" H 4900 7000 50  0000 L CNN
 F 1 "100nF" H 4900 6800 50  0000 L CNN
-F 2 "pkl_dipol:C_0402" H 4888 6750 50  0001 C CNN
+F 2 "Capacitor_SMD:C_0402_1005Metric" H 4888 6750 50  0001 C CNN
 F 3 "" H 4850 6900 50  0001 C CNN
 F 4 "1276-1002-1-ND" H -1050 -50 50  0001 C CNN "SN-DK"
@@
 F 0 "C86" H 5300 6250 50  0000 L CNN
 F 1 "10nF" H 5300 6050 50  0000 L CNN
-F 2 "pkl_dipol:C_0402" H 5288 6000 50  0001 C CNN
+F 2 "Capacitor_SMD:C_0402_1005Metric" H 5288 6000 50  0001 C CNN
 F 3 "" H 5250 6150 50  0001 C CNN
 F 4 "1276-1002-1-ND" H -650 -800 50  0001 C CNN "SN-DK"
@@
 F 0 "C87" H 5300 7000 50  0000 L CNN
 F 1 "10nF" H 5300 6800 50  0000 L CNN
-F 2 "pkl_dipol:C_0402" H 5288 6750 50  0001 C CNN
+F 2 "Capacitor_SMD:C_0402_1005Metric" H 5288 6750 50  0001 C CNN
 F 3 "" H 5250 6900 50  0001 C CNN
 F 4 "1276-1002-1-ND" H -650 -50 50  0001 C CNN "SN-DK"
@@
 F 0 "C88" H 5850 6250 50  0000 L CNN
 F 1 "100nF" H 5850 6050 50  0000 L CNN
-F 2 "pkl_dipol:C_0402" H 5838 6000 50  0001 C CNN
+F 2 "Capacitor_SMD:C_0402_1005Metric" H 5838 6000 50  0001 C CNN
 F 3 "" H 5800 6150 50  0001 C CNN
 F 4 "1276-1002-1-ND" H -100 -800 50  0001 C CNN "SN-DK"
@@
 F 0 "C89" H 5850 7000 50  0000 L CNN
 F 1 "100nF" H 5850 6800 50  0000 L CNN
-F 2 "pkl_dipol:C_0402" H 5838 6750 50  0001 C CNN
+F 2 "Capacitor_SMD:C_0402_1005Metric" H 5838 6750 50  0001 C CNN
 F 3 "" H 5800 6900 50  0001 C CNN
 F 4 "1276-1002-1-ND" H -100 -50 50  0001 C CNN "SN-DK"
@@
 F 0 "C90" H 6250 6250 50  0000 L CNN
 F 1 "10nF" H 6250 6050 50  0000 L CNN
-F 2 "pkl_dipol:C_0402" H 6238 6000 50  0001 C CNN
+F 2 "Capacitor_SMD:C_0402_1005Metric" H 6238 6000 50  0001 C CNN
 F 3 "" H 6200 6150 50  0001 C CNN
 F 4 "1276-1002-1-ND" H 300 -800 50  0001 C CNN "SN-DK"
@@
 F 0 "C91" H 6250 7000 50  0000 L CNN
 F 1 "10nF" H 6250 6800 50  0000 L CNN
-F 2 "pkl_dipol:C_0402" H 6238 6750 50  0001 C CNN
+F 2 "Capacitor_SMD:C_0402_1005Metric" H 6238 6750 50  0001 C CNN
 F 3 "" H 6200 6900 50  0001 C CNN
 F 4 "1276-1002-1-ND" H 300 -50 50  0001 C CNN "SN-DK"
@@
 F 0 "C100" H 9165 3896 50  0000 L CNN
 F 1 "10nF" H 9165 3805 50  0000 L CNN
-F 2 "pkl_dipol:C_0402" H 9088 3700 50  0001 C CNN
+F 2 "Capacitor_SMD:C_0402_1005Metric" H 9088 3700 50  0001 C CNN
 F 3 "~" H 9050 3850 50  0001 C CNN
 F 4 "Samsung Electro-Mechanics" H 0   0   50  0001 C CNN "Mfg"

Commit message: hw.r0_3: Update schematics with 85F-5G symbol
Parts:
- removed U3: ECP5U25, gkl_housings_bga:caBGA_381_17x17, symbol gkl_lattice:ECP5U25-BG381
- added U2: ECP5UM5G_85_CABGA381, gkl_housings_bga:caBGA_381_17x17, symbol ECP5UM5G-85Pinout:ECP5UM5G_85_CABGA381
Connections:
- net labels removed: +1V1, +2V5, PORT0_VCCIO, PORT1_VCCIO, PORT2_VCCIO
- wire segments 77 -> 54
Other:
- moved on the sheet: C100, C80, C81, C82, C83, C84, C85, C86, C87, C88, C89, C90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

Commit message: hw.r0_3: Start pin assignments for DDR3
Parts:
- added R70: 51R, Resistor_SMD:R_0402_1005Metric, symbol Device:R
- added U6: S25FL127S, Package_SO:SOIJ-8_5.3x5.3mm_P1.27mm, symbol gkl_mem:AT25SF081
- U2: symbol ECP5UM5G-85Pinout:ECP5UM5G_85_CABGA381 -> gkl_lattice:ECP5UM5G_85_CABGA381
Connections:
- net labels added: 1v1, 2v5, CFG.CLK, CFG.CS, CFG.IO0, CFG.IO1, CFG.IO2, CFG.IO3, TCK, TDI, TDO, TMS
- wire segments 54 -> 85
Other:
- moved on the sheet: C100, R4
