File: hardware/ButterStick_r0.3/TestPonts.kicad_sch (KiCad schematic)
At the start: 24 parts

Commit message: hw.r0_3: major blocks roughly routed
Parts:
- removed TP1, TP14, TP15, TP16, TP17, TP18, TP19, TP2, TP20, TP21, TP22, TP23, TP24, TP25, TP26, TP27, TP28, TP29, TP3, TP30, TP4, TP5, TP6, TP7: SMD_TESTPONT, TestPoint:TestPoint_Pad_D1.0mm, symbol Connector:TestPoint_Flag
