File: hardware/ButterStick_r1.0/ButterStick.kicad_sch (KiCad schematic)
At the start: 12 parts

Commit message: hw.r1d0: Update BOM fieids in schematic.
Parts:
- FID1, FID2, FID3, FID4, FID5, FID6, H1, H2, LOGO2: PN (none) -> DNP
- R1: Mfg Stackpole Electronics Inc -> Yageo; PN RMCF0402FT210K -> RC0402FR-07210KL
- R2: Mfg Stackpole Electronics Inc -> Yageo; PN RMCF0402FT84K5 -> RC0402FR-0784K5L
- R3: Mfg Stackpole Electronics Inc -> Yageo; PN RMCF0402FT49K9 -> RC0402FR-0749K9L
Changed lines of the file:
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@@
     (comment 2 "SYZYGY compatible")
   )
+  (bus_alias "RGMII" (members "RESET" "MDC" "MDIO" "TX[0..3]" "RX[0..3]" "TX_CTRL" "TX_CLK" "RX_CTRL" "RX_CLK" "INT" "CLK125"))
+  (bus_alias "I2C" (members "SDA" "SCL"))
   (bus_alias "SYZYGY_STD" (members "D0_P" "D0_N" "D2_P" "D2_N" "D4_P" "D4_N" "D6_P" "D6_N" "S16" "S18" "S20" "S22" "S24" "S26" "P2C_CLK_P" "P2C_CLK_N" "VIO1" "R_GA" "D1_P" "D1_N" "D3_P" "D3_N" "D5_P" "D5_N" "D7_P" "D7_N" "S17" "S19" "S21" "S23" "S25" "S27" "C2P_CLK_P" "C2P_CLK_N"))
-  (bus_alias "I2C" (members "SDA" "SCL"))
   (bus_alias "SYZYGY_TXR4" (members "RX0_P" "RX0_N" "RX1_P" "RX1_N" "REFCLK_P" "REFCLK_N" "S2" "S4" "S6" "S8" "RX3_P" "RX3_N" "RX2_P" "RX2_N" "P2C_CLK_P" "P2C_CLK_N" "VIO1" "R_GA" "TX0_P" "TX0_N" "TX1_P" "TX1_N" "S0" "S1" "S3" "S5" "S7" "S9" "TX3_P" "TX3_N" "TX2_P" "TX2_N" "C2P_CLK_P" "C2P_CLK_N"))
   (bus_alias "ULPI" (members "DATA[0..7]" "STP" "NXT" "DIR" "RESET" "REFCLK"))
+  (bus_alias "DRAM_CTRL" (members "A[15..0]" "BA[2..0]" "LDM" "UDM" "ODT[0..1]" "RAS" "CAS" "WE" "CK0_P" "CK0_N" "CKE[0..1]" "CS[0..1]" "CK1_N" "CK1_P" "RST"))
   (bus_alias "DRAM_DAT" (members "DQ[15..0]" "LDQS_P" "LDQS_N" "UDQS_P" "UDQS_N"))
   (bus_alias "SDMMC" (members "DAT[0..3]" "CMD" "CK" "CD"))
-  (bus_alias "RGMII" (members "RESET" "MDC" "MDIO" "TX[0..3]" "RX[0..3]" "TX_CTRL" "TX_CLK" "RX_CTRL" "RX_CLK" "INT" "CLK125"))
-  (bus_alias "DRAM_CTRL" (members "A[15..0]" "BA[2..0]" "LDM" "UDM" "ODT[0..1]" "RAS" "CAS" "WE" "CK0_P" "CK0_N" "CKE[0..1]" "CS[0..1]" "CK1_N" "CK1_P" "RST"))
   (junction (at 180.34 105.41) (diameter 0) (color 0 0 0 0))
   (junction (at 180.34 124.46) (diameter 0) (color 0 0 0 0))
@@
     (stroke (width 0) (type solid) (color 0 0 0 0))
   )
-  (bus (pts (xy 182.88 90.17) (xy 182.88 119.38))
-    (stroke (width 0) (type solid) (color 0 0 0 0))
-  )
-  (bus (pts (xy 182.88 119.38) (xy 182.88 154.94))
+  (bus (pts (xy 182.88 90.17) (xy 182.88 100.33))
+    (stroke (width 0) (type solid) (color 0 0 0 0))
+  )
+  (bus (pts (xy 182.88 100.33) (xy 182.88 138.43))
+    (stroke (width 0) (type solid) (color 0 0 0 0))
+  )
+  (bus (pts (xy 182.88 138.43) (xy 182.88 154.94))
     (stroke (width 0) (type solid) (color 0 0 0 0))
   )
@@
       (effects (font (size 1.27 1.27)) hide)
     )
+    (property "PN" "DNP" (id 4) (at 266.7 185.42 0)
+      (effects (font (size 1.27 1.27)) hide)
+    )
   )
   (symbol (lib_id "Mechanical:Fiducial") (at 269.24 182.88 0) (unit 1)
@@
       (effects (font (size 1.27 1.27)) hide)
     )
+    (property "PN" "DNP" (id 4) (at 269.24 182.88 0)
+      (effects (font (size 1.27 1.27)) hide)
+    )
   )
   (symbol (lib_id "Mechanical:Fiducial") (at 271.78 185.42 0) (unit 1)
@@
       (effects (font (size 1.27 1.27)) hide)
     )
+    (property "PN" "DNP" (id 4) (at 271.78 185.42 0)
+      (effects (font (size 1.27 1.27)) hide)
+    )
   )
   (symbol (lib_id "Mechanical:Fiducial") (at 276.86 185.42 0) (unit 1)
@@
       (effects (font (size 1.27 1.27)) hide)
     )
+    (property "PN" "DNP" (id 4) (at 276.86 185.42 0)
+      (effects (font (size 1.27 1.27)) hide)
+    )
   )
   (symbol (lib_id "Mechanical:Fiducial") (at 279.4 182.88 0) (unit 1)
@@
       (effects (font (size 1.27 1.27)) hide)
     )
+    (property "PN" "DNP" (id 4) (at 279.4 182.88 0)
+      (effects (font (size 1.27 1.27)) hide)
+    )
   )
   (symbol (lib_id "Mechanical:Fiducial") (at 281.94 185.42 0) (unit 1)
@@
     )
     (property "Datasheet" "~" (id 3) (at 281.94 185.42 0)
+      (effects (font (size 1.27 1.27)) hide)
+    )
+    (property "PN" "DNP" (id 4) (at 281.94 185.42 0)
       (effects (font (size 1.27 1.27)) hide)
     )
@@
       (effects (font (size 1.27 1.27)) hide)
     )
+    (property "PN" "DNP" (id 4) (at 271.78 168.91 0)
+      (effects (font (size 1.27 1.27)) hide)
+    )
   )
   (symbol (lib_id "Mechanical:MountingHole") (at 276.86 168.91 0) (unit 1)
@@
       (effects (font (size 1.27 1.27)) hide)
     )
+    (property "PN" "DNP" (id 4) (at 276.86 168.91 0)
+      (effects (font (size 1.27 1.27)) hide)
+    )
   )
   (symbol (lib_name "Device:R_1") (lib_id "Device:R") (at 236.22 110.49 90) (unit 1)
@@
       (effects (font (size 1.27 1.27)) hide)
     )
-    (property "Mfg" "Stackpole Electronics Inc" (id 4) (at 334.01 336.55 0)
-      (effects (font (size 1.27 1.27)) hide)
-    )
-    (property "PN" "RMCF0402FT210K" (id 5) (at 334.01 336.55 0)
+    (property "Mfg" "Yageo" (id 4) (at 334.01 336.55 0)
+      (effects (font (size 1.27 1.27)) hide)
+    )
+    (property "PN" "RC0402FR-07210KL" (id 5) (at 334.01 336.55 0)
       (effects (font (size 1.27 1.27)) hide)
     )
@@
       (effects (font (size 1.27 1.27)) hide)
     )
-    (property "Mfg" "Stackpole Electronics Inc" (id 4) (at 328.93 342.9 0)
-      (effects (font (size 1.27 1.27)) hide)
-    )
-    (property "PN" "RMCF0402FT84K5" (id 5) (at 328.93 342.9 0)
+    (property "Mfg" "Yageo" (id 4) (at 328.93 342.9 0)
+      (effects (font (size 1.27 1.27)) hide)
+    )
+    (property "PN" "RC0402FR-0784K5L" (id 5) (at 328.93 342.9 0)
       (effects (font (size 1.27 1.27)) hide)
     )
@@
       (effects (font (size 1.27 1.27)) hide)
     )
-    (property "Mfg" "Stackpole Electronics Inc" (id 4) (at 330.2 375.92 0)
-      (effects (font (size 1.27 1.27)) hide)
-    )
-    (property "PN" "RMCF0402FT49K9" (id 5) (at 330.2 375.92 0)
+    (property "Mfg" "Yageo" (id 4) (at 330.2 375.92 0)
+      (effects (font (size 1.27 1.27)) hide)
+    )
+    (property "PN" "RC0402FR-0749K9L" (id 5) (at 330.2 375.92 0)
       (effects (font (size 1.27 1.27)) hide)
     )
@@
       (effects (font (size 1.27 1.27)) hide)
     )
+    (property "PN" "DNP" (id 4) (at 264.16 173.99 0)
+      (effects (font (size 1.27 1.27)) hide)
+    )
   )
   (sheet (at 130.81 138.43) (size 40.64 12.7)
@@
     )
   )
-  (sheet (at 184.15 40.64) (size 33.02 16.51)
-    (stroke (width 0.1524) (type solid) (color 132 0 132 1))
-    (fill (color 255 255 255 1.0000))
-    (property "Sheet name" "sheetPower" (id 0) (at 184.15 40.0045 0)
+  (sheet (at 184.15 44.45) (size 33.02 12.7)
+    (stroke (width 0.1524) (type solid) (color 132 0 132 1))
+    (fill (color 255 255 255 1.0000))
+    (property "Sheet name" "sheetPower" (id 0) (at 184.15 43.8145 0)
       (effects (font (size 1.27 1.27)) (justify left bottom))
     )
@@
     )
     (path "/8f8777ba-89bc-4499-bd4b-cc705875169a/6e9f50fc-0d6d-4629-99f0-7a47156cbe46"
-      (reference "L1") (unit 1)
+      (reference "FB6") (unit 1)
     )
     (path "/8f8777ba-89bc-4499-bd4b-cc705875169a/611fe4c8-c48a-4856-9e02-e00324abcd11"
-      (reference "L2") (unit 1)
+      (reference "FB7") (unit 1)
     )
     (path "/8f8777ba-89bc-4499-bd4b-cc705875169a/4f09c2c4-c9b4-46e7-a4eb-6a4b16a5a140"
