File: hardware/ButterStick_r1.0/fileFPGA.kicad_sch (KiCad schematic)
At the start: 67 parts, among them J6 Conn_01x06_Male, U4 ECP5UM5G_85_CABGA381, U5 S25FL127S

Commit message: hw.r1d0: Review complete, gerbers generated
Connections:
- net P_1V2_A renamed P_1V1_A
- net P_1V2_T renamed P_1V1_T
Other:
- moved on the sheet: C122, C123, C124, C125, C126, C127, C128, C129, C130, C131, C132, C133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

Commit message: hw.r1d0: Update BOM fieids in schematic.
Parts:
- C122, C123, C124, C125, C126, C127, C132, C133, C134, C135, C136, C137: Mfg (none) -> Yageo; PN (none) -> CC0402KRX5R5BB474
- C128, C129, C130, C131: value 10nF -> 0.01uF; Mfg (none) -> Yageo; PN (none) -> CC0402KRX7R8BB103
- C138, C139, C60, C62: Mfg (none) -> Yageo; PN (none) -> CC0402MRX5R6BB475
- C140, C141, C58, C59: Field4 4V -> (none); Mfg (none) -> Murata Electronics; PN (none) -> GRM188R60G476ME15D; Tol (none) -> 4V
- C156, C32, C42, C44, C46, C48, C50: Mfg Samsung Electro-Mechanics -> Yageo; PN CL05B103KP5NNNC -> CC0402KRX5R6BB104; SN-DK 1276-1002-1-ND -> (none); Tol (none) -> 10V / X5R
- C20: Mfg Samsung Electro-Mechanics -> Yageo; PN CL05B103KP5NNNC -> CC0402KRX5R6BB104; Tol (none) -> 10V / X5R
- C30, C43, C45, C47, C49, C51: Mfg Samsung Electro-Mechanics -> Yageo; PN CL05B104KP5NNNC -> CC0402KRX5R5BB474; SN-DK 1276-1002-1-ND -> (none)
- C38, C39, C40, C52, C53, C56, C63, C66, C67, C70, C71: Mfg Samsung Electro-Mechanics -> Yageo; PN CL05B104KP5NNNC -> CC0402KRX5R6BB104; SN-DK 1276-1002-1-ND -> (none); Tol (none) -> 10V / X5R
- C65, C72: Mfg (none) -> Yageo; PN CL10A106MP8NNNC -> CC0603KRX5R5BB106; SN-DK 445-7486-1-ND -> (none)
- FB1, FB2, FB3, FB4: footprint Capacitor_SMD:C_0603_1608Metric -> Inductor_SMD:L_0603_1608Metric; Mfg (none) -> TDK Corporation; PN (none) -> MPZ1608D101BTA00
- J6: PN (none) -> DNP
- R45, R55: Mfg Stackpole Electronics Inc -> Yageo; PN RC0402JR-074K7L -> RC0402FR-074K7L; SN-DK P10KDECT-ND -> (none)
- R46, R49, R50: Mfg Stackpole Electronics Inc -> Yageo; PN RC0402JR-074K7L -> DNP; SN-DK P10KDECT-ND -> (none)
- R47, R48, R51: Mfg Stackpole Electronics Inc -> Yageo; PN RC0402JR-074K7L -> RC0402FR-071KL; SN-DK P10KDECT-ND -> (none)
- R52: Mfg Stackpole Electronics Inc -> Yageo; PN RC0402JR-074K7L -> RC0402FR-0751RL; SN-DK P10KDECT-ND -> (none)
- U4: Mfg (none) -> Lattice Semiconductor Corporation; PN (none) -> LFE5UM5G-85F-8BG381C; manf# ECP5UM5G_85 -> (none)
- U5: value S25FL127S -> W25Q128JVSIQ; Mfg Cypress Semiconductor Corp -> Winbond Electronics; PN S25FL127SABMFI101 -> W25Q128JVSIQ; SN-DK 1092-1178-1-ND -> (none)

Commit message: hw.r1d0: Fix RGMII straps
This commit correctly sets the stop resistos on the RGMII lines to 1K5
instead of DNP.
Also regenerate and add a schematic in PDF format.

Fixes #6
Parts:
- C138, C139, C60, C62: Mfg Yageo -> (none); PN CC0402MRX5R6BB475 -> CC0402KRX5R6BB475
- C140, C141, C58, C59: value 47uF -> 22uF; Mfg Murata Electronics -> Yageo; PN GRM188R60G476ME15D -> CC0603MRX5R5BB226; Tol 4V -> 6.3V
- R46, R49, R50: Mfg Yageo -> (none); PN DNP -> (none)
- U4: PN LFE5UM5G-85F-8BG381C -> LFE5UM5G-85F-8BG381I

Commit message: hardware.r1d0: Update BOM values in schematic
Regenerate schematics and export BOM

Fixes #9
Connections:
- net +1V1 renamed P_1V2_FPGA
- net P_1V1_A renamed P_1V2_A
- net P_1V1_T renamed P_1V2_T
Changed lines of the file:
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@@
 (kicad_sch (version 20201015) (generator eeschema)
-  (page 1 18)
   (paper "A4")
   (title_block
     (title "ButterStick")
-    (date "2020-11-01")
+    (date "2021-01-10")
     (rev "r1.0")
     (company "GsD")
@@
   (no_connect (at 162.56 107.95))
   (no_connect (at 85.09 106.68))
+  (no_connect (at 162.56 110.49))
   (no_connect (at 85.09 104.14))
-  (no_connect (at 162.56 110.49))
   (bus_entry (at 29.21 43.18) (size -2.54 -2.54)
     (stroke (width 0.1524) (type solid) (color 0 0 0 0))
@@
     (effects (font (size 1.27 1.27)) (justify left bottom))
   )
-  (global_label "P_1V1_A" (shape input) (at 109.22 45.72 180)
+  (global_label "P_1V2_A" (shape input) (at 109.22 45.72 180)    (property "Intersheet References" "${INTERSHEET_REFS}" (id 0) (at 98.7388 45.6406 0)
+      (effects (font (size 1.27 1.27)) (justify right) hide)
+    )
     (effects (font (size 1.27 1.27)) (justify right))
   )
-  (global_label "P_1V1_T" (shape input) (at 250.19 22.86 0)
+  (global_label "P_1V2_FPGA" (shape input) (at 176.53 146.05 90)    (property "Intersheet References" "${INTERSHEET_REFS}" (id 0) (at 176.4506 131.9402 90)
+      (effects (font (size 1.27 1.27)) (justify left) hide)
+    )
     (effects (font (size 1.27 1.27)) (justify left))
   )
-  (global_label "P_1V1_T" (shape input) (at 250.19 43.18 0)
+  (global_label "P_1V2_FPGA" (shape input) (at 203.2 77.47 90)    (property "Intersheet References" "${INTERSHEET_REFS}" (id 0) (at 203.1206 63.3602 90)
+      (effects (font (size 1.27 1.27)) (justify left) hide)
+    )
+    (effects (font (size 1.27 1.27)) (justify left))
+  )
+  (global_label "P_1V2_T" (shape input) (at 250.19 22.86 0)    (property "Intersheet References" "${INTERSHEET_REFS}" (id 0) (at 260.5503 22.7806 0)
+      (effects (font (size 1.27 1.27)) (justify left) hide)
+    )
+    (effects (font (size 1.27 1.27)) (justify left))
+  )
+  (global_label "P_1V2_T" (shape input) (at 250.19 43.18 0)    (property "Intersheet References" "${INTERSHEET_REFS}" (id 0) (at 260.5503 43.1006 0)
+      (effects (font (size 1.27 1.27)) (justify left) hide)
+    )
     (effects (font (size 1.27 1.27)) (justify left))
   )
@@
     )
   )
-  (symbol (lib_id "gkl_power:+1V1") (at 176.53 146.05 0) (unit 1)
-    (in_bom yes) (on_board yes)
-    (property "Reference" "#PWR099" (id 0) (at 176.53 149.86 0)
-      (effects (font (size 1.27 1.27)) hide)
-    )
-    (property "Value" "+1V1" (id 1) (at 176.6062 142.2146 0))
-    (property "Footprint" "" (id 2) (at 176.53 146.05 0)
-      (effects (font (size 1.27 1.27)) hide)
-    )
-    (property "Datasheet" "" (id 3) (at 176.53 146.05 0)
-      (effects (font (size 1.27 1.27)) hide)
-    )
-  )
   (symbol (lib_id "gkl_power:+2V5") (at 180.34 77.47 0) (unit 1)
     (in_bom yes) (on_board yes)
@@
       (effects (font (size 1.27 1.27)) hide)
     )
-  )
-  (symbol (lib_id "gkl_power:+1V1") (at 203.2 77.47 0) (unit 1)
-    (in_bom yes) (on_board yes)
-    (property "Reference" "#PWR071" (id 0) (at 203.2 81.28 0)
-      (effects (font (size 1.27 1.27)) hide)
-    )
-    (property "Value" "+1V1" (id 1) (at 203.2762 73.6346 0))
-    (property "Footprint" "" (id 2) (at 203.2 77.47 0)
-      (effects (font (size 1.27 1.27)) hide)
-    )
-    (property "Datasheet" "" (id 3) (at 203.2 77.47 0)
-      (effects (font (size 1.27 1.27)) hide)
-    )

Commit message: hardware.r1d0: Tidy up BOM entries
Export HTML Interactive BOM
Parts:
- C138, C139, C60, C62: Mfg (none) -> Yageo
- J6: now left out of the parts list
- R46, R49, R50: PN (none) -> DNP
Changed lines of the file:
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@@
   (junction (at 257.81 114.3) (diameter 1.016) (color 0 0 0 0))
   (junction (at 257.81 124.46) (diameter 1.016) (color 0 0 0 0))
-  (no_connect (at 162.56 107.95))
   (no_connect (at 85.09 106.68))
+  (no_connect (at 162.56 107.95))
   (no_connect (at 162.56 110.49))
   (no_connect (at 85.09 104.14))
@@
       (effects (font (size 1.27 1.27)) hide)
     )
-    (property "PN" "" (id 5) (at -218.44 156.21 0)
+    (property "PN" "DNP" (id 5) (at -218.44 156.21 0)
       (effects (font (size 1.27 1.27)) hide)
     )
@@
       (effects (font (size 1.27 1.27)) hide)
     )
-    (property "PN" "" (id 5) (at -214.63 171.45 0)
+    (property "PN" "DNP" (id 5) (at -214.63 171.45 0)
       (effects (font (size 1.27 1.27)) hide)
     )
@@
       (effects (font (size 1.27 1.27)) hide)
     )
-    (property "PN" "" (id 5) (at -210.82 156.21 0)
+    (property "PN" "DNP" (id 5) (at -210.82 156.21 0)
       (effects (font (size 1.27 1.27)) hide)
     )
@@
       (effects (font (size 1.27 1.27)) hide)
     )
+    (property "Mfg" "Yageo" (id 4) (at 127 29.21 0)
+      (effects (font (size 1.27 1.27)) hide)
+    )
   )
   (symbol (lib_name "Device:C_16") (lib_id "Device:C") (at 127 50.8 0) (unit 1)
@@
       (effects (font (size 1.27 1.27)) hide)
     )
+    (property "Mfg" "Yageo" (id 4) (at 127 50.8 0)
+      (effects (font (size 1.27 1.27)) hide)
+    )
   )
   (symbol (lib_name "Device:C_20") (lib_id "Device:C") (at 134.62 29.21 0) (unit 1)
@@
       (effects (font (size 1.27 1.27)) hide)
     )
+    (property "Mfg" "Yageo" (id 4) (at 232.41 27.94 0)
+      (effects (font (size 1.27 1.27)) hide)
+    )
   )
   (symbol (lib_name "Device:C_2") (lib_id "Device:C") (at 232.41 48.26 0) (mirror y) (unit 1)
@@
       (effects (font (size 1.27 1.27)) hide)
     )
+    (property "Mfg" "Yageo" (id 4) (at 232.41 48.26 0)
+      (effects (font (size 1.27 1.27)) hide)
+    )
   )
   (symbol (lib_id "Device:C") (at 233.68 152.4 0) (unit 1)
@@
   )
   (symbol (lib_id "Connector:Conn_01x06_Male") (at 134.62 170.18 0) (mirror y) (unit 1)
-    (in_bom yes) (on_board yes)
+    (in_bom no) (on_board yes)
     (property "Reference" "J6" (id 0) (at 135.3313 170.8594 0)
       (effects (font (size 1.27 1.27)) (justify right))

Commit message: Fix RGB G/B signals
- Corrects a mistake where blue and green signals were swapped
- Regenerate schematic

Closes #12
Parts:
- C140, C141, C58, C59: PN CC0603MRX5R5BB226 -> (none)
