File: hardware/ButterStick_r1.0/fileIO.kicad_sch (KiCad schematic)
At the start: 9 parts, among them J2 MicroSD, SW1 SW_Push, SW2 SW_Push, U3 PUSB3FR6

Commit message: hw.r1d0: Update BOM fieids in schematic.
Parts:
- C64: Mfg Samsung Electro-Mechanics -> Yageo; PN CL05B104KP5NNNC -> CC0402KRX5R6BB104; SN-DK 1276-1002-1-ND -> (none); Tol (none) -> 10V / X5R
- C69: Mfg (none) -> Yageo; PN CL10A106MP8NNNC -> CC0603KRX5R5BB106; SN-DK 445-7486-1-ND -> (none)
- FB5: footprint Capacitor_SMD:C_0603_1608Metric -> Inductor_SMD:L_0603_1608Metric; Mfg (none) -> TDK Corporation; PN (none) -> MPZ1608D101BTA00
- J2: Mfg (none) -> Molex; SN-DK WM6357CT-ND -> (none)
- R33, R34: Mfg (none) -> Yageo; PN (none) -> RC0402FR-0710KL
- SW1, SW2: Mfg (none) -> C&K; PN (none) -> PTS810SJK250SMTRLFS
- U3: MFG Nexperia USA Inc. -> (none); Mfg (none) -> Nexperia USA Inc.
Changed lines of the file:
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@@
 (kicad_sch (version 20200618) (host eeschema "5.99.0-unknown-73168a9~101~ubuntu18.04.1")
-  (page 4 18)
+  (page 1 18)
   (paper "A4")
   (title_block
@@
       (effects (font (size 1.27 1.27)) hide)
     )
+    (property "Mfg" "Yageo" (id 4) (at 219.71 85.09 0)
+      (effects (font (size 1.27 1.27)) hide)
+    )
+    (property "PN" "RC0402FR-0710KL" (id 4) (at 219.71 85.09 0)
+      (effects (font (size 1.27 1.27)) hide)
+    )
   )
   (symbol (lib_id "Device:R") (at 223.52 85.09 0) (unit 1)
@@
       (effects (font (size 1.27 1.27)) hide)
     )
+    (property "Mfg" "Yageo" (id 4) (at 223.52 85.09 0)
+      (effects (font (size 1.27 1.27)) hide)
+    )
+    (property "PN" "RC0402FR-0710KL" (id 4) (at 223.52 85.09 0)
+      (effects (font (size 1.27 1.27)) hide)
+    )
   )
   (symbol (lib_id "Device:Ferrite_Bead_Small") (at 129.54 66.04 90) (unit 1)
@@
     (property "Reference" "FB5" (id 0) (at 129.54 60.128 90))
     (property "Value" "100R" (id 1) (at 129.54 62.4267 90))
-    (property "Footprint" "Capacitor_SMD:C_0603_1608Metric" (id 2) (at 129.54 67.818 90)
+    (property "Footprint" "Inductor_SMD:L_0603_1608Metric" (id 2) (at 129.54 67.818 90)
       (effects (font (size 1.27 1.27)) hide)
     )
     (property "Datasheet" "~" (id 3) (at 129.54 66.04 0)
+      (effects (font (size 1.27 1.27)) hide)
+    )
+    (property "Mfg" "TDK Corporation" (id 4) (at 129.54 66.04 0)
+      (effects (font (size 1.27 1.27)) hide)
+    )
+    (property "PN" "MPZ1608D101BTA00" (id 5) (at 129.54 66.04 0)
       (effects (font (size 1.27 1.27)) hide)
     )
@@
       (effects (font (size 1.27 1.27)) hide)
     )
-    (property "SN-DK" "1276-1002-1-ND" (id 4) (at 270.51 214.63 0)
-      (effects (font (size 1.27 1.27)) hide)
-    )
-    (property "PN" "CL05B104KP5NNNC" (id 5) (at 270.51 214.63 0)
-      (effects (font (size 1.27 1.27)) hide)
-    )
-    (property "Mfg" "Samsung Electro-Mechanics" (id 6) (at 311.15 312.42 0)
+    (property "SN-DK" "" (id 4) (at 270.51 214.63 0)
+      (effects (font (size 1.27 1.27)) hide)
+    )
+    (property "PN" "CC0402KRX5R6BB104" (id 5) (at 270.51 214.63 0)
+      (effects (font (size 1.27 1.27)) hide)
+    )
+    (property "Mfg" "Yageo" (id 6) (at 311.15 312.42 0)
+      (effects (font (size 1.27 1.27)) hide)
+    )
+    (property "Tol" "10V / X5R" (id 4) (at 144.78 66.04 0)
       (effects (font (size 1.27 1.27)) hide)
     )
@@
       (effects (font (size 1.27 1.27)) hide)
     )
-    (property "SN-DK" "445-7486-1-ND" (id 4) (at 280.67 102.87 0)
-      (effects (font (size 1.27 1.27)) hide)
-    )
-    (property "PN" "CL10A106MP8NNNC" (id 5) (at 259.08 332.74 0)
+    (property "SN-DK" "" (id 4) (at 280.67 102.87 0)
+      (effects (font (size 1.27 1.27)) hide)
+    )
+    (property "PN" "CC0603KRX5R5BB106" (id 5) (at 259.08 332.74 0)
+      (effects (font (size 1.27 1.27)) hide)
+    )
+    (property "Mfg" "Yageo" (id 4) (at 144.78 71.12 0)
       (effects (font (size 1.27 1.27)) hide)
     )
@@
       (effects (font (size 1.27 1.27)) hide)
     )
+    (property "Mfg" "C&K" (id 4) (at 232.41 93.98 0)
+      (effects (font (size 1.27 1.27)) hide)
+    )
+    (property "PN" "PTS810SJK250SMTRLFS" (id 5) (at 232.41 93.98 0)
+      (effects (font (size 1.27 1.27)) hide)
+    )
   )
   (symbol (lib_id "Switch:SW_Push") (at 232.41 104.14 0) (unit 1)
@@
       (effects (font (size 1.27 1.27)) hide)
     )
+    (property "Mfg" "C&K" (id 4) (at 232.41 104.14 0)
+      (effects (font (size 1.27 1.27)) hide)
+    )
+    (property "PN" "PTS810SJK250SMTRLFS" (id 5) (at 232.41 104.14 0)
+      (effects (font (size 1.27 1.27)) hide)
+    )
   )
   (symbol (lib_id "Connector:Conn_01x11_Male") (at 157.48 92.71 0) (mirror y) (unit 1)
@@
       (effects (font (size 1.27 1.27)) hide)
     )
-    (property "SN-DK" " WM6357CT-ND" (id 4) (at 157.48 92.71 0)
+    (property "SN-DK" "" (id 4) (at 157.48 92.71 0)
       (effects (font (size 1.524 1.524)) hide)
     )
     (property "PN" "1040310811" (id 5) (at 300.99 190.5 0)
+      (effects (font (size 1.27 1.27)) hide)
+    )
+    (property "Mfg" "Molex" (id 4) (at 157.48 92.71 0)
       (effects (font (size 1.27 1.27)) hide)
     )
@@
       (effects (font (size 1.27 1.27)) hide)
     )
-    (property "MFG" "Nexperia USA Inc." (id 4) (at 214.63 -40.64 0)
+    (property "MFG" "" (id 4) (at 214.63 -40.64 0)
       (effects (font (size 1.27 1.27)) hide)
     )
@@
       (effects (font (size 1.27 1.27)) hide)
     )
+    (property "Mfg" "Nexperia USA Inc." (id 4) (at 125.73 110.49 0)
+      (effects (font (size 1.27 1.27)) hide)
+    )

Commit message: hw.r1d0: Fix RGMII straps
This commit correctly sets the stop resistos on the RGMII lines to 1K5
instead of DNP.
Also regenerate and add a schematic in PDF format.

Fixes #6
Changed lines of the file:
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@@
-(kicad_sch (version 20200618) (host eeschema "5.99.0-unknown-73168a9~101~ubuntu18.04.1")
+(kicad_sch (version 20201015) (generator eeschema)
   (page 1 18)
   (paper "A4")
   (title_block
     (title "ButterStick")
-    (date "2020-07-17")
+    (date "2020-11-01")
     (rev "r1.0")
     (company "GsD")
     (comment 1 "Functional prototyping board for the Lattice ECP5.")
-  )
-  (junction (at 119.38 97.79) (diameter 0) (color 0 0 0 0))
-  (junction (at 121.92 95.25) (diameter 0) (color 0 0 0 0))
-  (junction (at 124.46 90.17) (diameter 0) (color 0 0 0 0))
-  (junction (at 127 85.09) (diameter 0) (color 0 0 0 0))
-  (junction (at 129.54 82.55) (diameter 0) (color 0 0 0 0))
-  (junction (at 132.08 80.01) (diameter 0) (color 0 0 0 0))
-  (junction (at 138.43 66.04) (diameter 0) (color 0 0 0 0))
-  (junction (at 138.43 71.12) (diameter 0) (color 0 0 0 0))
-  (junction (at 138.43 100.33) (diameter 0) (color 0 0 0 0))
-  (junction (at 138.43 102.87) (diameter 0) (color 0 0 0 0))
-  (junction (at 151.13 71.12) (diameter 0) (color 0 0 0 0))
-  (junction (at 219.71 78.74) (diameter 0) (color 0 0 0 0))
-  (junction (at 219.71 93.98) (diameter 0) (color 0 0 0 0))
-  (junction (at 223.52 104.14) (diameter 0) (color 0 0 0 0))
-  (junction (at 241.3 104.14) (diameter 0) (color 0 0 0 0))
-  (junction (at 132.08 36.83) (diameter 0) (color 0 0 0 0))
+    (comment 2 "SYZYGY compatible")
+  )
+  (junction (at 119.38 97.79) (diameter 1.016) (color 0 0 0 0))
+  (junction (at 121.92 95.25) (diameter 1.016) (color 0 0 0 0))
+  (junction (at 124.46 90.17) (diameter 1.016) (color 0 0 0 0))
+  (junction (at 127 85.09) (diameter 1.016) (color 0 0 0 0))
+  (junction (at 129.54 82.55) (diameter 1.016) (color 0 0 0 0))
+  (junction (at 132.08 80.01) (diameter 1.016) (color 0 0 0 0))
+  (junction (at 138.43 66.04) (diameter 1.016) (color 0 0 0 0))
+  (junction (at 138.43 71.12) (diameter 1.016) (color 0 0 0 0))
+  (junction (at 138.43 100.33) (diameter 1.016) (color 0 0 0 0))
+  (junction (at 138.43 102.87) (diameter 1.016) (color 0 0 0 0))
+  (junction (at 151.13 71.12) (diameter 1.016) (color 0 0 0 0))
+  (junction (at 219.71 78.74) (diameter 1.016) (color 0 0 0 0))
+  (junction (at 219.71 93.98) (diameter 1.016) (color 0 0 0 0))
+  (junction (at 223.52 104.14) (diameter 1.016) (color 0 0 0 0))
+  (junction (at 241.3 104.14) (diameter 1.016) (color 0 0 0 0))
+  (junction (at 132.08 36.83) (diameter 1.016) (color 0 0 0 0))
   (bus_entry (at 100.33 77.47) (size 2.54 2.54)
     (stroke (width 0.1524) (type solid) (color 0 0 0 0))
@@
     (stroke (width 0) (type solid) (color 0 0 0 0))
   )
-  (bus (pts (xy 100.33 76.2) (xy 100.33 80.01))
+  (bus (pts (xy 100.33 76.2) (xy 100.33 77.47))
+    (stroke (width 0) (type solid) (color 0 0 0 0))
+  )
+  (bus (pts (xy 100.33 77.47) (xy 100.33 80.01))
     (stroke (width 0) (type solid) (color 0 0 0 0))
   )
@@
     (stroke (width 0) (type solid) (color 0 0 0 0))
   )
-  (bus (pts (xy 100.33 82.55) (xy 100.33 90.17))
-    (stroke (width 0) (type solid) (color 0 0 0 0))
-  )
-  (bus (pts (xy 100.33 90.17) (xy 100.33 95.25))
+  (bus (pts (xy 100.33 82.55) (xy 100.33 87.63))
+    (stroke (width 0) (type solid) (color 0 0 0 0))
+  )
+  (bus (pts (xy 100.33 87.63) (xy 100.33 90.17))
+    (stroke (width 0) (type solid) (color 0 0 0 0))
+  )
+  (bus (pts (xy 100.33 90.17) (xy 100.33 92.71))
+    (stroke (width 0) (type solid) (color 0 0 0 0))
+  )
+  (bus (pts (xy 100.33 92.71) (xy 100.33 95.25))
     (stroke (width 0) (type solid) (color 0 0 0 0))
   )
@@
     (stroke (width 0) (type solid) (color 0 0 0 0))
   )
-  (bus (pts (xy 134.62 36.83) (xy 134.62 41.91))
-    (stroke (width 0) (type solid) (color 0 0 0 0))
-  )
+  (bus (pts (xy 134.62 36.83) (xy 134.62 39.37))
+    (stroke (width 0) (type solid) (color 0 0 0 0))
+  )
+  (bus (pts (xy 134.62 39.37) (xy 134.62 41.91))
+    (stroke (width 0) (type solid) (color 0 0 0 0))
+  )
